File: Hardware/cape.sch (EAGLE design)
At the start: 102 parts, among them IC1 RT7258, IC2 RT7258, IC3 74HC125, J1 JST-BM07B-GHS-TBT, J10 JST-BM07B-GHS-TBT, J11 JST-BM07B-GHS-TBT, J12 JST-BM07B-GHS-TBT, J13 JST-BM07B-GHS-TBT, J14 JST-BM07B-GHS-TBT, J15 JST-BM07B-GHS-TBT, J16 JST-BM07B-GHS-TBT, J17 JST-BM07B-GHS-TBT, J18 JST-BM07B-GHS-TBT, J19 JST-BM07B-GHS-TBT, J2 JST-BM07B-GHS-TBT, J20 JST-BM07B-GHS-TBT, J21 JST-BM07B-GHS-TBT, J22 JST-BM07B-GHS-TBT, J23 JST-BM07B-GHS-TBT, J24 JST-BM07B-GHS-TBT, J25 JST-BM07B-GHS-TBT, J26 JST-BM07B-GHS-TBT, J27 JST-BM07B-GHS-TBT, J28 JST-BM07B-GHS-TBT, J29 JST-BM07B-GHS-TBT, J3 JST-BM07B-GHS-TBT, J30 JST-BM07B-GHS-TBT, J31 JST-BM07B-GHS-TBT, J32 JST-BM07B-GHS-TBT, J4 JST-BM07B-GHS-TBT, J5 JST-BM07B-GHS-TBT, J6 JST-BM07B-GHS-TBT, J7 JST-BM07B-GHS-TBT, J8 JST-BM07B-GHS-TBT, J9 JST-BM07B-GHS-TBT, Q1 FDS6670, Q2 FDS6670, X1 RJ45-6L2-B, X2 RJ45-6L2-B

Commit message: Updated cape schematic and library, added datasheets
Parts:
- removed C13, C14: 22uF, SparkFun-Capacitors:CAP1206
- removed C15, C16: 47uF, SparkFun-Capacitors:CAP1206
- removed C18: 10uF, SparkFun-Capacitors:CAP1206
- removed C6, C7, C8: 1uF, SparkFun-Capacitors:CAP1206
- removed FX1: TG110-E055N5, halo-electronics:TG110-E055N5
- removed IC2: RT7258, TotU:RT7258
- removed J10, J11, J12, J13, J14, J15, J16, J17, J18, J19, J20, J21, J22, J23, J24, J25, J26, J27, J28, J29, J3, J30, J31, J32, J4, J5, J6, J7, J8, J9: JST-BM07B-GHS-TBT, TotU:JST-BM07B-GHS-TBT
- removed L2: MURATA_INDUCTOR_3900, TotU:MURATA_INDUCTOR_3900
- removed Q2: FDS6670, TotU:FDS6670
- removed R26, R27, R28, R29, R30, R31, R32, R33, R34, R35, R36, R37, R38: (no value), SparkFun-Passives:RESISTOR0805-RES
- removed R39, R40: 10k, SparkFun-Passives:RESISTOR1206
- removed R4: 100k, SparkFun-Passives:RESISTOR1206
- removed R5: 62k, SparkFun-Passives:RESISTOR1206
- removed R6: 20k, SparkFun-Passives:RESISTOR1206
- added C20, C21: 1uF, SparkFun-Capacitors:CAP1206
- added C22, C23: 10uF, SparkFun-Capacitors:CAP1206
- added IC4, IC5: 74VHC541, cape:74VHC541
- C5: value 22uF -> 10uF
- J1, J2: value JST-BM07B-GHS-TBT -> FCI-10118064-5001310LF; device TotU:JST-BM07B-GHS-TBT -> cape:FCI-10118064-5001310LF
- R10, R11, R12, R13, R14, R15, R16, R17, R18, R19, R20, R21, R22, R23, R24, R25, R7, R8, R9: device SparkFun-Passives:RESISTOR0805-RES -> resistor:R-US_M0805
Connections:
- removed net LED-1: J1.7, R7.1
- removed net LED-10: J10.7, R12.1
- removed net LED-11: J11.7, R13.1
- removed net LED-12: J12.7, R14.1
- removed net LED-13: J13.7, R19.1
- removed net LED-14: J14.7, R20.1
- removed net LED-15: J15.7, R21.1
- removed net LED-16: J16.7, R22.1
- removed net LED-17: J17.7, R23.1
- removed net LED-18: J18.7, R24.1
- removed net LED-19: J19.7, R25.1
- removed net LED-2: J2.7, R8.1
- removed net LED-20: J20.7, R26.1
- removed net LED-21: J21.7, R31.1
- removed net LED-22: J22.7, R32.1
- removed net LED-23: J23.7, R33.1
- removed net LED-24: J24.7, R34.1
- removed net LED-25: J25.7, R27.1
- removed net LED-26: J26.7, R28.1
- removed net LED-27: J27.7, R29.1
- removed net LED-28: J28.7, R30.1
- removed net LED-29: J29.7, R35.1
- removed net LED-3: J3.7, R9.1
- removed net LED-30: J30.7, R36.1
- removed net LED-31: J31.7, R37.1
- removed net LED-32: J32.7, R38.1
- removed net LED-4: J4.7, R10.1
- removed net LED-5: J5.7, R15.1
- removed net LED-6: J6.7, R16.1
- removed net LED-7: J7.7, R17.1
- removed net LED-8: J8.7, R18.1
- removed net LED-9: J9.7, R11.1
- removed net N$10: C7.1, IC2.EN, R4.1
- removed net N$11: C8.1, IC2.BOOT
- removed net N$12: C8.2, IC2.SW, L2.1, Q2.D
- removed net N$14: IC2.FB, R5.1, R6.2
- removed net N$15: IC2.BG, Q2.G
- removed net N$9: C6.1, IC2.VCC
- removed net RD+: FX1.3, X2.3
- removed net RD-: FX1.1, X2.6
- removed net SCL: IC3.1Y, J1.2, J10.2, J11.2, J12.2, J13.2, J14.2, J15.2, J16.2, J17.2, J18.2, J19.2, J2.2, J20.2, J21.2, J22.2, J23.2, J24.2, J25.2, J26.2, J27.2, J28.2, J29.2, J3.2, J30.2, J31.2, J32.2, J4.2, J5.2, J6.2, J7.2, J8.2, J9.2
- removed net SDI-1: J1.1, U$1.UART2_RXD
- removed net SDI-10: J10.1, U$1.UART1_RXD
- removed net SDI-11: J11.1, U$1.UART1_TXD
- removed net SDI-12: J12.1, U$1.CLKOUT2
- removed net SDI-13: J13.1, U$1.EHRPWM2A
- removed net SDI-14: J14.1, U$1.EHRPWM2B
- removed net SDI-15: J15.1, U$1.GPIO0_26
- removed net SDI-16: J16.1, U$1.GPIO0_27
- removed net SDI-17: J17.1, U$1.UART4_RXD
- removed net SDI-18: J18.1, U$1.UART4_TXD
- removed net SDI-19: J19.1, U$1.GPIO1_12
- removed net SDI-2: J2.1, U$1.UART2_TXD
- removed net SDI-20: J20.1, U$1.GPIO1_13
- removed net SDI-21: J21.1, U$1.GPIO1_14
- removed net SDI-22: J22.1, U$1.GPIO1_15
- removed net SDI-23: J23.1, U$1.GPIO1_16
- removed net SDI-24: J24.1, U$1.GPIO1_17
- removed net SDI-25: J25.1, U$1.EHRPWM1A
- removed net SDI-26: J26.1, U$1.EHRPWM1B
- removed net SDI-27: J27.1, U$1.GPIO1_28
- removed net SDI-28: J28.1, U$1.GPIO1_29
- removed net SDI-29: J29.1, U$1.GPIO2_1
- removed net SDI-3: J3.1, U$1.I2C1_SDA
- removed net SDI-30: J30.1, U$1.TIMER4
- removed net SDI-31: J31.1, U$1.TIMER7
- removed net SDI-32: J32.1, U$1.TIMER6
- removed net SDI-4: J4.1, U$1.I2C1_SCL
- removed net SDI-5: J5.1, U$1.GPIO0_7
- removed net SDI-6: J6.1, U$1.UART4_CTSN
- removed net SDI-7: J7.1, U$1.UART4_RTSN
- removed net SDI-8: J8.1, U$1.UART5_CTSN
- removed net SDI-9: J9.1, U$1.UART5_RTSN
- removed net TD+: FX1.8, X2.1
- removed net TD-: FX1.6, X2.2
- new net AD0: IC4.A8, U$1.GPIO1_0
- new net AD1: IC4.A7, U$1.GPIO1_1
- new net AD10: IC5.A6, U$1.GPIO0_26
- new net AD11: IC5.A5, U$1.GPIO0_27
- new net AD12: IC5.A4, U$1.GPIO1_12
- new net AD13: IC5.A3, U$1.GPIO1_13
- new net AD14: IC5.A2, U$1.GPIO1_14
- new net AD15: IC5.A1, U$1.GPIO1_15
- new net AD2: IC4.A6, U$1.GPIO1_2
- new net AD3: IC4.A5, U$1.GPIO1_3
- new net AD4: IC4.A4, U$1.GPIO1_4
- new net AD5: IC4.A3, U$1.GPIO1_5
- new net AD6: IC4.A2, U$1.GPIO1_6
- new net AD7: IC4.A1, U$1.GPIO1_7
- new net AD8: IC5.A8, U$1.EHRPWM2A
- new net AD9: IC5.A7, U$1.EHRPWM2B
- new net BKL0: J1.A6
- new net BLK1: J1.B6
- new net BLK10: J2.C6
- new net BLK11: J2.D6
- new net BLK12: J2.E6
- new net BLK13: J2.F6
- new net BLK14: J2.G6
- new net BLK15: J2.H6
- new net BLK2: J1.C6
- new net BLK3: J1.D6
- new net BLK4: J1.E6
- new net BLK5: J1.F6
- new net BLK6: J1.G6
- new net BLK7: J1.H6
- new net BLK8: J2.A6
- new net BLK9: J2.B6
- new net DATA0: J1.A1, R14.2
- new net DATA1: J1.B1, R13.2
- new net DATA10: J2.C1, R20.2
- new net DATA11: J2.D1, R19.2
- new net DATA12: J2.E1, R18.2
- new net DATA13: J2.F1, R17.2
- new net DATA14: J2.G1, R16.2
- new net DATA15: J2.H1, R15.2
- new net DATA2: J1.C1, R12.2
- new net DATA3: J1.D1, R11.2
- new net DATA4: J1.E1, R10.2
- new net DATA5: J1.F1, R9.2
- new net DATA6: J1.G1, R8.2
- new net DATA7: J1.H1, R7.2
- new net DATA8: J2.A1, R22.2
- new net DATA9: J2.B1, R21.2
- new net N$13: IC4.Y3, R9.1
- new net N$16: IC4.Y4, R10.1
- new net N$17: IC4.Y5, R11.1
- new net N$18: IC4.Y6, R12.1
- new net N$19: IC4.Y7, R13.1
- new net N$20: IC4.Y8, R14.1
- new net N$21: IC5.Y1, R15.1
- new net N$22: IC5.Y2, R16.1
- new net N$23: IC5.Y3, R17.1
- new net N$24: IC5.Y4, R18.1
- new net N$25: IC5.Y5, R19.1
- new net N$26: IC5.Y6, R20.1
- new net N$27: IC5.Y7, R21.1
- new net N$28: IC5.Y8, R22.1
- new net N$29: IC3.3Y, R25.1
- new net N$30: IC3.2Y, R24.1
- new net N$31: IC3.1Y, R23.1
- new net N$5: IC4.Y1, R7.1
- new net N$6: IC4.Y2, R8.1
- new net SCK: J1.A8, J1.B8, J1.C8, J1.D8, J1.E8, J1.F8, J1.G8, J1.H8, J2.A8, J2.B8, J2.C8, J2.D8, J2.E8, J2.F8, J2.G8, J2.H8, R23.2
- net DC: now also J1.A4, J1.B4, J1.C4, J1.D4, J1.E4, J1.F4, J1.G4, J1.H4, J2.A4, J2.B4, J2.C4, J2.D4, J2.E4, J2.F4, J2.G4, J2.H4, R24.2; no longer IC3.2Y, J1.3, J10.3, J11.3, J12.3, J13.3, J14.3, J15.3, J16.3, J17.3, J18.3, J19.3, J2.3, J20.3, J21.3, J22.3, J23.3, J24.3, J25.3, J26.3, J27.3, J28.3, J29.3, J3.3, J30.3, J31.3, J32.3, J4.3, J5.3, J6.3, J7.3, J8.3, J9.3
- net DC_RAW: now also U$1.GPIO1_29; no longer U$1.TIMER5
- net GND: now also C20.2, C21.2, C22.2, C23.2, C5.1, IC4.G1, IC4.G2, IC4.GND, IC5.G1, IC5.G2, IC5.GND, J1.A2, J1.A7, J1.B2, J1.B7, J1.C2, J1.C7, J1.D2, J1.D7, J1.E2, J1.E7, J1.F2, J1.F7, J1.G2, J1.G7, J1.H2, J1.H7, J2.A2, J2.A7, J2.B2, J2.B7, J2.C2, J2.C7, J2.D2, J2.D7, J2.E2, J2.E7, J2.F2, J2.F7, J2.G2, J2.G7, J2.H2, J2.H7; no longer C13.2, C14.2, C15.2, C16.2, C18.2, C5.2, C6.2, C7.2, FX1.15, IC2.GND, J1.4, J10.4, J11.4, J12.4, J13.4, J14.4, J15.4, J16.4, J17.4, J18.4, J19.4, J2.4, J20.4, J21.4, J22.4, J23.4, J24.4, J25.4, J26.4, J27.4, J28.4, J29.4, J3.4, J30.4, J31.4, J32.4, J4.4, J5.4, J6.4, J7.4, J8.4, J9.4, Q2.S, R40.1, R6.1
- net RST: now also J1.A5, J1.B5, J1.C5, J1.D5, J1.E5, J1.F5, J1.G5, J1.H5, J2.A5, J2.B5, J2.C5, J2.D5, J2.E5, J2.F5, J2.G5, J2.H5, R25.2; no longer IC3.3Y, J1.5, J10.5, J11.5, J12.5, J13.5, J14.5, J15.5, J16.5, J17.5, J18.5, J19.5, J2.5, J20.5, J21.5, J22.5, J23.5, J24.5, J25.5, J26.5, J27.5, J28.5, J29.5, J3.5, J30.5, J31.5, J32.5, J4.5, J5.5, J6.5, J7.5, J8.5, J9.5
- net RST_RAW: now also U$1.GPIO1_31; no longer R39.1, R40.2, U$1.GPIO2_7
- net RX+: now also X2.3; no longer FX1.14
- net RX-: now also X2.6; no longer FX1.16
- net SCL_RAW: now also U$1.TIMER6; no longer U$1.GPIO2_6
- net TX+: now also X2.1; no longer FX1.9
- net TX-: now also X2.2; no longer FX1.11
- net VCC3V3: now also C20.1, C21.1, C22.1, C23.1, C5.2, IC4.VCC, IC5.VCC, J1.A3, J1.B3, J1.C3, J1.D3, J1.E3, J1.F3, J1.G3, J1.H3, J2.A3, J2.B3, J2.C3, J2.D3, J2.E3, J2.F3, J2.G3, J2.H3, U$1.VDD_3V3EXP@2; no longer C13.1, C14.1, C15.1, C16.1, J1.6, J10.6, J11.6, J12.6, J13.6, J14.6, J15.6, J16.6, J17.6, J18.6, J19.6, J2.6, J20.6, J21.6, J22.6, J23.6, J24.6, J25.6, J26.6, J27.6, J28.6, J29.6, J3.6, J30.6, J31.6, J32.6, J4.6, J5.6, J6.6, J7.6, J8.6, J9.6, L2.2, R39.2, R5.2
- net VCC5V: no longer C18.1, C5.1, IC2.VIN, R10.2, R11.2, R12.2, R13.2, R14.2, R15.2, R16.2, R17.2, R18.2, R19.2, R20.2, R21.2, R22.2, R23.2, R24.2, R25.2, R26.2, R27.2, R28.2, R29.2, R30.2, R31.2, R32.2, R33.2, R34.2, R35.2, R36.2, R37.2, R38.2, R4.2, R7.2, R8.2, R9.2
- net VIN: no longer FX1.10
Other:
- note removed: "5v -> 3.3v Step Down"
- note removed: "DNP"
- moved on the sheet: C5, R10, R11, R12, R13, R14, R15, R16, R17, R18, R19, R20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

Commit message: Working on board routing
Parts:
- removed C19: 1uF, SparkFun-Capacitors:CAP1206
- removed C5: 10uF, SparkFun-Capacitors:CAP1206
- removed IC3: 74HC125, TotU:74HC125
- removed R23, R24, R25: (no value), resistor:R-US_M0805
- added C6: 1uF, SparkFun-Capacitors:CAP1206
- added C7: 10uF, SparkFun-Capacitors:CAP1206
- added IC2: 74VHC541, cape:74VHC541
- added Q2, Q3, Q4, Q5, Q6, Q7, Q8, Q9: N-MOSFET-DUAL, cape:N-MOSFET-DUAL
- added R26, R27, R28, R29, R30, R4, R5, R6: (no value), resistor:R-US_M0805
- J1, J2: PARTNO (none) -> 10118064-5001310LF
Connections:
- removed net BKL0: J1.A6
- removed net BLK1: J1.B6
- removed net BLK10: J2.C6
- removed net BLK11: J2.D6
- removed net BLK12: J2.E6
- removed net BLK13: J2.F6
- removed net BLK14: J2.G6
- removed net BLK15: J2.H6
- removed net BLK2: J1.C6
- removed net BLK3: J1.D6
- removed net BLK4: J1.E6
- removed net BLK5: J1.F6
- removed net BLK6: J1.G6
- removed net BLK7: J1.H6
- removed net BLK8: J2.A6
- removed net BLK9: J2.B6
- removed net DC: J1.A4, J1.B4, J1.C4, J1.D4, J1.E4, J1.F4, J1.G4, J1.H4, J2.A4, J2.B4, J2.C4, J2.D4, J2.E4, J2.F4, J2.G4, J2.H4, R24.2
- removed net N$29: IC3.3Y, R25.1
- removed net N$30: IC3.2Y, R24.1
- removed net N$31: IC3.1Y, R23.1
- removed net RST_RAW: IC3.3A, U$1.GPIO1_31
- removed net SCK: J1.A8, J1.B8, J1.C8, J1.D8, J1.E8, J1.F8, J1.G8, J1.H8, J2.A8, J2.B8, J2.C8, J2.D8, J2.E8, J2.F8, J2.G8, J2.H8, R23.2
- new net BL0: J1.A6, Q6G$1.D
- new net BL1: J1.B6, Q6G$2.D
- new net BL10: J2.C6, Q3G$1.D
- new net BL11: J2.D6, Q3G$2.D
- new net BL12: J2.E6, Q4G$1.D
- new net BL13: J2.F6, Q4G$2.D
- new net BL14: J2.G6, Q5G$1.D
- new net BL15: J2.H6, Q5G$2.D
- new net BL2: J1.C6, Q7G$1.D
- new net BL3: J1.D6, Q7G$2.D
- new net BL4: J1.E6, Q8G$1.D
- new net BL5: J1.F6, Q8G$2.D
- new net BL6: J1.G6, Q9G$1.D
- new net BL7: J1.H6, Q9G$2.D
- new net BL8: J2.A6, Q2G$1.D
- new net BL9: J2.B6, Q2G$2.D
- new net DC0: J1.A4, J1.B4, J1.C4, J1.D4, R27.2
- new net DC1: J1.E4, J1.F4, J1.G4, J1.H4, R28.2
- new net DC2: J2.A4, J2.B4, J2.C4, J2.D4, R29.2
- new net DC3: J2.E4, J2.F4, J2.G4, J2.H4, R30.2
- new net N$10: IC2.Y2, R5.1
- new net N$11: IC2.Y3, R6.1
- new net N$12: IC2.Y4, R26.1
- new net N$14: IC2.Y5, R27.1
- new net N$15: IC2.Y6, R28.1
- new net N$32: IC2.Y7, R29.1
- new net N$33: IC2.Y8, R30.1
- new net N$9: IC2.Y1, R4.1
- new net PRU0-0: Q2G$1.G, U$1.SPI1_SCLK
- new net PRU0-1: Q2G$2.G, U$1.SPI1_DO
- new net PRU0-2: Q3G$1.G, U$1.SPI1_DI
- new net PRU0-3: Q3G$2.G, U$1.SPI1_CS0
- new net PRU0-4: Q4G$1.G, U$1.GPIO0_7
- new net PRU0-5: Q4G$2.G, U$1.GPIO3_19
- new net PRU0-6: Q5G$1.G, U$1.CLKOUT2
- new net PRU0-7: Q5G$2.G, U$1.GPIO3_21
- new net PRU1-0: Q6G$1.G, U$1.GPIO2_6
- new net PRU1-1: Q6G$2.G, U$1.GPIO2_7
- new net PRU1-10: U$1.GPIO2_24
- new net PRU1-12: U$1.GPIO1_30
- new net PRU1-2: Q7G$1.G, U$1.GPIO2_8
- new net PRU1-3: Q7G$2.G, U$1.GPIO2_9
- new net PRU1-4: Q8G$1.G, U$1.GPIO2_10
- new net PRU1-5: Q8G$2.G, U$1.GPIO2_11
- new net PRU1-6: Q9G$1.G, U$1.GPIO2_12
- new net PRU1-7: Q9G$2.G, U$1.GPIO2_13
- new net PRU1-8: U$1.GPIO2_22
- new net PRU1-9: U$1.GPIO2_23
- new net SCK0: J1.A8, J1.B8, J1.C8, J1.D8, R4.2
- new net SCK1: J1.E8, J1.F8, J1.G8, J1.H8, R5.2
- new net SCK2: J2.A8, J2.B8, J2.C8, J2.D8, R26.2
- new net SCK3: J2.E8, J2.F8, J2.G8, J2.H8, R6.2
- net DC_RAW: now also IC2.A5, IC2.A6, IC2.A7, IC2.A8; no longer IC3.2A
- net GND: now also C6.2, C7.2, IC2.G1, IC2.G2, IC2.GND, Q2G$1.S, Q2G$2.S, Q3G$1.S, Q3G$2.S, Q4G$1.S, Q4G$2.S, Q5G$1.S, Q5G$2.S, Q6G$1.S, Q6G$2.S, Q7G$1.S, Q7G$2.S, Q8G$1.S, Q8G$2.S, Q9G$1.S, Q9G$2.S; no longer C19.1, C5.1, IC3.1OE, IC3.2OE, IC3.3OE, IC3.4A, IC3.4OE, IC3.GND
- net RST: now also U$1.GPIO1_31; no longer R25.2
- net SCL_RAW: now also IC2.A1, IC2.A2, IC2.A3, IC2.A4; no longer IC3.1A
- net VCC3V3: now also C6.1, C7.1, IC2.VCC; no longer C19.2, C5.2, IC3.VCC
- net VCC5V: now also U$1.VDD_5V@2

Commit message: Routing
Parts:
- removed X1, X2: RJ45-6L2-B, con-tycoelectronics:RJ45-6L2-B
- added J3, J4: RJ45-8P8C, cape:RJ45-8P8C
Connections:
- removed net RX+: X1.3, X2.3
- removed net RX-: X1.6, X2.6
- removed net TX+: X1.1, X2.1
- removed net TX-: X1.2, X2.2
- new net RX_N: J3.6, J4.6
- new net RX_P: J3.3, J4.3
- new net TX_N: J3.2, J4.2
- new net TX_P: J3.1, J4.1
- net GND: now also J3.7, J3.8; no longer X1.7, X1.8, X1.S@1, X1.S@2, X1.S@3, X1.S@4, X2.S@1, X2.S@2, X2.S@3, X2.S@4
- net VIN: now also J3.4, J3.5; no longer X1.4, X1.5

Commit message: Finished v1 board
Parts:
- added 3V, 5V, GND, PRU1-10, PRU1-12, PRU1-8, PRU1-9, VIN: PTR1TP20R, tenna_avr_AD7021_v0_9_shrink:PTR1TP20R
- added F1: PTC, cape:PTC
- added U$4, U$5, U$6: FIDUCIAL, adafruit:FIDUCIAL
- C1, C10, C9: PARTNO (none) -> C3216X5R1V226M160AC
- C11, C12: PARTNO (none) -> C1206C476M8PACTU
- C17, C22, C23, C7: PARTNO (none) -> GMK316AB7106KL-TR
- C2, C20, C21, C3, C4, C6: PARTNO (none) -> C3216X7R1H105K160AB
- IC1: PARTNO (none) -> RT7258GSP
- IC2, IC4, IC5: PARTNO (none) -> 74VHC541FT(BE)
- J3, J4: PARTNO (none) -> 54602-908LF
- L1: value MURATA_INDUCTOR_3900 -> 2.8uH; PARTNO (none) -> 39H282C
- Q1: PARTNO (none) -> FDS6670AS
- R1: PARTNO (none) -> RC1206JR-07100KL
- R2: PARTNO (none) -> RC1206FR-0793K1L
- R3: PARTNO (none) -> ERJ-8ENF1802V
Connections:
- new net VFUSE: C1.1, C17.1, F1.1, IC1.VIN, R1.2
- net GND: now also GND.TP
- net PRU1-10: now also PRU1-10.TP
- net PRU1-12: now also PRU1-12.TP
- net PRU1-8: now also PRU1-8.TP
- net PRU1-9: now also PRU1-9.TP
- net VCC3V3: now also 3V.TP
- net VCC5V: now also 5V.TP
- net VIN: now also F1.2, VIN.TP; no longer C1.1, C17.1, IC1.VIN, R1.2

Commit message: Added resistors (resolves #3), changed mosfet package (resolves #6), changed power input
Parts:
- removed C1, C10, C9: 22uF, SparkFun-Capacitors:CAP1206
- removed C11, C12: 47uF, SparkFun-Capacitors:CAP1206
- removed C17: 10uF, SparkFun-Capacitors:CAP1206
- removed C2, C3, C4: 1uF, SparkFun-Capacitors:CAP1206
- removed F1: PTC, cape:PTC
- removed IC1: RT7258, TotU:RT7258
- removed J4: RJ45-8P8C, cape:RJ45-8P8C
- removed L1: 2.8uH, TotU:MURATA_INDUCTOR_3900
- removed Q1: FDS6670, TotU:FDS6670
- added R23, R24, R25, R31, R32, R33, R34, R35, R36, R37, R38, R39, R40: R18 1/2W, resistor:R-US_M0805
- J3: PARTNO 54602-908LF -> (none)
- Q2, Q3, Q4, Q5, Q6, Q7, Q8, Q9: value N-MOSFET-DUAL -> N-MOSFET-DUALSO8; device cape:N-MOSFET-DUAL -> cape:N-MOSFET-DUALSO8; PARTNO DMN3190LDW-7 -> *
- R1: value 100k -> R18 1/2W; device SparkFun-Passives:RESISTOR1206 -> resistor:R-US_M0805; PARTNO RC1206JR-07100KL -> (none)
- R2: value 93k -> R18 1/2W; device SparkFun-Passives:RESISTOR1206 -> resistor:R-US_M0805; PARTNO RC1206FR-0793K1L -> (none)
- R3: value 18k -> R18 1/2W; device SparkFun-Passives:RESISTOR1206 -> resistor:R-US_M0805; PARTNO ERJ-8ENF1802V -> (none)
Connections:
- removed net RX_N: J3.6, J4.6
- removed net RX_P: J3.3, J4.3
- removed net TX_N: J3.2, J4.2
- removed net TX_P: J3.1, J4.1
- removed net VFUSE: C1.1, C17.1, F1.1, IC1.VIN, R1.2
- new net N$29: Q9G$1.D, R31.2
- new net N$30: Q9G$2.D, R32.2
- new net N$31: Q2G$1.D, R33.2
- new net N$34: Q2G$2.D, R34.2
- new net N$35: Q3G$1.D, R35.2
- new net N$36: Q3G$2.D, R36.2
- new net N$37: Q4G$1.D, R37.2
- new net N$38: Q4G$2.D, R38.2
- new net N$39: Q5G$1.D, R39.2
- new net N$40: Q5G$2.D, R40.2
- net BL0: now also R1.1; no longer Q6G$1.D
- net BL1: now also R2.1; no longer Q6G$2.D
- net BL10: now also R35.1; no longer Q3G$1.D
- net BL11: now also R36.1; no longer Q3G$2.D
- net BL12: now also R37.1; no longer Q4G$1.D
- net BL13: now also R38.1; no longer Q4G$2.D
- net BL14: now also R39.1; no longer Q5G$1.D
- net BL15: now also R40.1; no longer Q5G$2.D
- net BL2: now also R3.1; no longer Q7G$1.D
- net BL3: now also R23.1; no longer Q7G$2.D
- net BL4: now also R24.1; no longer Q8G$1.D
- net BL5: now also R25.1; no longer Q8G$2.D
- net BL6: now also R31.1; no longer Q9G$1.D
- net BL7: now also R32.1; no longer Q9G$2.D
- net BL8: now also R33.1; no longer Q2G$1.D
- net BL9: now also R34.1; no longer Q2G$2.D
- net GND: now also J3.1, J3.3, J3.5; no longer C1.2, C10.2, C11.2, C12.2, C17.2, C2.2, C3.2, C9.2, IC1.GND, J3.8, Q1.S, R3.1
- net N$1: now also Q6G$1.D, R1.2; no longer C2.1, IC1.VCC
- net N$2: now also Q6G$2.D, R2.2; no longer C3.1, IC1.EN, R1.1
- net N$3: now also Q7G$1.D, R3.2; no longer C4.1, IC1.BOOT
- net N$4: now also Q7G$2.D, R23.2; no longer C4.2, IC1.SW, L1.1, Q1.D
- net N$7: now also Q8G$1.D, R24.2; no longer IC1.FB, R2.1, R3.2
- net N$8: now also Q8G$2.D, R25.2; no longer IC1.BG, Q1.G
- net VCC5V: now also J3.2, J3.4, J3.6, J3.8; no longer C10.1, C11.1, C12.1, C9.1, L1.2, R2.2
- net VIN: no longer F1.2, J3.4, J3.5
Other:
- note removed: "24v -> 5v Step Down"
- moved on the sheet: J3, R1, R2, R3
