File: Hardware/cape.sch (EAGLE design)
At the start: 72 parts, among them IC2 74VHC541, IC4 74VHC541, IC5 74VHC541, J1 FCI-10118064-5001310LF, J2 FCI-10118064-5001310LF, J3 RJ45-8P8C, Q2 N-MOSFET-DUALSO8, Q3 N-MOSFET-DUALSO8, Q4 N-MOSFET-DUALSO8, Q5 N-MOSFET-DUALSO8, Q6 N-MOSFET-DUALSO8, Q7 N-MOSFET-DUALSO8, Q8 N-MOSFET-DUALSO8, Q9 N-MOSFET-DUALSO8

Commit message: Started adding A/B switches and more ports
Parts:
- removed R1, R2, R23, R24, R25, R3, R31, R32, R33, R34, R35, R36, R37, R38, R39, R40: R18 1/2W, resistor:R-US_M0805
- removed R10, R11, R12, R13, R14, R15, R16, R17, R18, R19, R20, R21, R22, R26, R27, R28, R29, R30, R4, R5, R6, R7, R8, R9: (no value), resistor:R-US_M0805
- added C1, C4: 10uF, SparkFun-Capacitors:CAP1206
- added C2, C3: 1uF, SparkFun-Capacitors:CAP1206
- added U$7, U$8: SN74CBT16292DLRSSOP56, cape:SN74CBT16292DLRSSOP56
Connections:
- removed net N$10: IC2.Y2, R5.1
- removed net N$11: IC2.Y3, R6.1
- removed net N$12: IC2.Y4, R26.1
- removed net N$13: IC4.Y3, R9.1
- removed net N$14: IC2.Y5, R27.1
- removed net N$15: IC2.Y6, R28.1
- removed net N$16: IC4.Y4, R10.1
- removed net N$17: IC4.Y5, R11.1
- removed net N$18: IC4.Y6, R12.1
- removed net N$19: IC4.Y7, R13.1
- removed net N$20: IC4.Y8, R14.1
- removed net N$21: IC5.Y1, R15.1
- removed net N$22: IC5.Y2, R16.1
- removed net N$23: IC5.Y3, R17.1
- removed net N$24: IC5.Y4, R18.1
- removed net N$25: IC5.Y5, R19.1
- removed net N$26: IC5.Y6, R20.1
- removed net N$27: IC5.Y7, R21.1
- removed net N$28: IC5.Y8, R22.1
- removed net N$32: IC2.Y7, R29.1
- removed net N$33: IC2.Y8, R30.1
- removed net N$5: IC4.Y1, R7.1
- removed net N$6: IC4.Y2, R8.1
- removed net N$9: IC2.Y1, R4.1
- new net 10A: IC5.Y2, U$7.10A
- new net 11A: IC5.Y3, U$7.11A
- new net 12A: IC5.Y4, U$7.12A
- new net 13A: IC5.Y5, U$8.1A
- new net 14A: IC5.Y6, U$8.2A
- new net 15A: IC5.Y7, U$8.3A
- new net 16A: IC5.Y8, U$8.4A
- new net 17A: IC2.Y4, U$8.5A, U$8.6A
- new net 19A: IC2.Y5, U$8.7A, U$8.8A
- new net 1A: IC4.Y1, U$7.1A
- new net 21A: IC2.Y6, U$8.10A, U$8.9A
- new net 23A: IC2.Y7, U$8.11A, U$8.12A
- new net 2A: IC4.Y2, U$7.2A
- new net 3A: IC4.Y3, U$7.3A
- new net 4A: IC4.Y4, U$7.4A
- new net 5A: IC4.Y5, U$7.5A
- new net 6A: IC4.Y6, U$7.6A
- new net 7A: IC4.Y7, U$7.7A
- new net 8A: IC4.Y8, U$7.8A
- new net 9A: IC5.Y1, U$7.9A
- new net SCL_1: IC2.A2, IC2.A3, IC2.Y1
- new net SCL_2: IC2.A4, IC2.A5, IC2.Y2
- new net SCL_3: IC2.A6, IC2.A7, IC2.Y3
- net AD0: now also IC5.A8; no longer IC4.A8
- net AD1: now also IC5.A7; no longer IC4.A7
- net AD10: now also IC4.A8; no longer IC5.A6
- net AD11: now also IC5.A3; no longer IC5.A5
- net AD12: now also IC4.A6; no longer IC5.A4
- net AD13: now also IC4.A5; no longer IC5.A3
- net AD2: now also IC4.A3; no longer IC4.A6
- net AD3: now also IC4.A4; no longer IC4.A5
- net AD4: now also IC5.A6; no longer IC4.A4
- net AD5: now also IC5.A5; no longer IC4.A3
- net AD6: now also IC4.A1; no longer IC4.A2
- net AD7: now also IC4.A2; no longer IC4.A1
- net AD8: now also IC5.A4; no longer IC5.A8
- net AD9: now also IC4.A7; no longer IC5.A7
- net BL0: no longer R1.1
- net BL1: no longer R2.1
- net BL10: no longer R35.1
- net BL11: no longer R36.1
- net BL12: no longer R37.1
- net BL13: no longer R38.1
- net BL14: no longer R39.1
- net BL15: no longer R40.1
- net BL2: no longer R3.1
- net BL3: no longer R23.1
- net BL4: no longer R24.1
- net BL5: no longer R25.1
- net BL6: no longer R31.1
- net BL7: no longer R32.1
- net BL8: no longer R33.1
- net BL9: no longer R34.1
- net DATA0: no longer R14.2
- net DATA1: no longer R13.2
- net DATA10: no longer R20.2
- net DATA11: no longer R19.2
- net DATA12: no longer R18.2
- net DATA13: no longer R17.2
- net DATA14: no longer R16.2
- net DATA15: no longer R15.2
- net DATA2: no longer R12.2
- net DATA3: no longer R11.2
- net DATA4: no longer R10.2
- net DATA5: no longer R9.2
- net DATA6: no longer R8.2
- net DATA7: no longer R7.2
- net DATA8: no longer R22.2
- net DATA9: no longer R21.2
- net DC0: no longer R27.2
- net DC1: no longer R28.2
- net DC2: no longer R29.2
- net DC3: no longer R30.2
- net DC_RAW: no longer IC2.A5, IC2.A6, IC2.A7, IC2.A8
- net GND: now also C1.2, C2.2, C3.2, C4.2, U$7.GND, U$8.GND
- net N$1: no longer R1.2
- net N$2: no longer R2.2
- net N$29: no longer R31.2
- net N$3: no longer R3.2
- net N$30: no longer R32.2
- net N$31: no longer R33.2
- net N$34: no longer R34.2
- net N$35: no longer R35.2
- net N$36: no longer R36.2
- net N$37: no longer R37.2
- net N$38: no longer R38.2
- net N$39: no longer R39.2
- net N$4: no longer R23.2
- net N$40: no longer R40.2
- net N$7: no longer R24.2
- net N$8: no longer R25.2
- net SCK0: no longer R4.2
- net SCK1: no longer R5.2
- net SCK2: no longer R26.2
- net SCK3: no longer R6.2
- net SCL_RAW: no longer IC2.A2, IC2.A3, IC2.A4
- net VCC5V: now also C1.1, C2.1, C3.1, C4.1, U$7.VCC, U$8.VCC
Other:
- moved on the sheet: 3V, 5V, GND, PRU1-10, PRU1-12, PRU1-8, PRU1-9, U$1, VIN

Commit message: Work on routing A/B and mosfets
Parts:
- removed 3V, 5V, GND, PRU1-10, PRU1-12, PRU1-8, PRU1-9, VIN: PTR1TP20R, tenna_avr_AD7021_v0_9_shrink:PTR1TP20R
- removed C22, C23, C7: 10uF, SparkFun-Capacitors:CAP1206
- removed J1, J2: FCI-10118064-5001310LF, cape:FCI-10118064-5001310LF
- added Q1, Q10, Q11, Q12, Q13, Q14, Q15, Q16: N-MOSFET-DUALSO8, cape:N-MOSFET-DUALSO8
- added U$10, U$9: RJ45-8P8C-16FCI-16, cape:RJ45-8P8C-16FCI-16
- C1, C4: device SparkFun-Capacitors:CAP1206 -> SparkFun-Capacitors:CAP0805; PARTNO GMK316AB7106KL-TR -> (none)
- C2, C20, C21, C3, C6: device SparkFun-Capacitors:CAP1206 -> SparkFun-Capacitors:CAP0805; PARTNO C3216X7R1H105K160AB -> (none)
Connections:
- removed net BL0: J1.A6
- removed net BL1: J1.B6
- removed net BL10: J2.C6
- removed net BL11: J2.D6
- removed net BL12: J2.E6
- removed net BL13: J2.F6
- removed net BL14: J2.G6
- removed net BL15: J2.H6
- removed net BL2: J1.C6
- removed net BL3: J1.D6
- removed net BL4: J1.E6
- removed net BL5: J1.F6
- removed net BL6: J1.G6
- removed net BL7: J1.H6
- removed net BL8: J2.A6
- removed net BL9: J2.B6
- removed net DATA0: J1.A1
- removed net DATA1: J1.B1
- removed net DATA10: J2.C1
- removed net DATA11: J2.D1
- removed net DATA12: J2.E1
- removed net DATA13: J2.F1
- removed net DATA14: J2.G1
- removed net DATA15: J2.H1
- removed net DATA2: J1.C1
- removed net DATA3: J1.D1
- removed net DATA4: J1.E1
- removed net DATA5: J1.F1
- removed net DATA6: J1.G1
- removed net DATA7: J1.H1
- removed net DATA8: J2.A1
- removed net DATA9: J2.B1
- removed net DC0: J1.A4, J1.B4, J1.C4, J1.D4
- removed net DC1: J1.E4, J1.F4, J1.G4, J1.H4
- removed net DC2: J2.A4, J2.B4, J2.C4, J2.D4
- removed net DC3: J2.E4, J2.F4, J2.G4, J2.H4
- removed net N$1: Q6G$1.D
- removed net N$2: Q6G$2.D
- removed net N$29: Q9G$1.D
- removed net N$3: Q7G$1.D
- removed net N$30: Q9G$2.D
- removed net N$31: Q2G$1.D
- removed net N$34: Q2G$2.D
- removed net N$35: Q3G$1.D
- removed net N$36: Q3G$2.D
- removed net N$37: Q4G$1.D
- removed net N$38: Q4G$2.D
- removed net N$39: Q5G$1.D
- removed net N$4: Q7G$2.D
- removed net N$40: Q5G$2.D
- removed net N$7: Q8G$1.D
- removed net N$8: Q8G$2.D
- removed net PRU0-0: Q2G$1.G, U$1.SPI1_SCLK
- removed net PRU0-1: Q2G$2.G, U$1.SPI1_DO
- removed net PRU0-2: Q3G$1.G, U$1.SPI1_DI
- removed net PRU0-3: Q3G$2.G, U$1.SPI1_CS0
- removed net PRU0-4: Q4G$1.G, U$1.GPIO0_7
- removed net PRU0-5: Q4G$2.G, U$1.GPIO3_19
- removed net PRU0-6: Q5G$1.G, U$1.CLKOUT2
- removed net PRU0-7: Q5G$2.G, U$1.GPIO3_21
- removed net PRU1-0: Q6G$1.G, U$1.GPIO2_6
- removed net PRU1-1: Q6G$2.G, U$1.GPIO2_7
- removed net PRU1-10: PRU1-10.TP, U$1.GPIO2_24
- removed net PRU1-12: PRU1-12.TP, U$1.GPIO1_30
- removed net PRU1-2: Q7G$1.G, U$1.GPIO2_8
- removed net PRU1-3: Q7G$2.G, U$1.GPIO2_9
- removed net PRU1-4: Q8G$1.G, U$1.GPIO2_10
- removed net PRU1-5: Q8G$2.G, U$1.GPIO2_11
- removed net PRU1-6: Q9G$1.G, U$1.GPIO2_12
- removed net PRU1-7: Q9G$2.G, U$1.GPIO2_13
- removed net PRU1-8: PRU1-8.TP, U$1.GPIO2_22
- removed net PRU1-9: PRU1-9.TP, U$1.GPIO2_23
- removed net SCK0: J1.A8, J1.B8, J1.C8, J1.D8
- removed net SCK1: J1.E8, J1.F8, J1.G8, J1.H8
- removed net SCK2: J2.A8, J2.B8, J2.C8, J2.D8
- removed net SCK3: J2.E8, J2.F8, J2.G8, J2.H8
- removed net VIN: VIN.TP
- new net BL-0-1: Q2G$1.D, U$10G$9.6
- new net BL-0-2: Q2G$2.D, U$10G$1.6
- new net BL-1-1: Q3G$1.D, U$10G$10.6
- new net BL-1-2: Q3G$2.D, U$10G$2.6
- new net BL-10-1: U$9G$8.6
- new net BL-10-2: U$9G$16.6
- new net BL-11-1: Q7G$1.D, U$10G$14.6
- new net BL-11-2: Q7G$2.D, U$10G$6.6
- new net BL-12-2: U$9G$14.6
- new net BL-13-1: U$9G$5.6
- new net BL-13-2: U$9G$13.6
- new net BL-14-1: Q8G$1.D, U$10G$15.6
- new net BL-14-2: Q8G$2.D, U$10G$7.6
- new net BL-15-1: Q9G$1.D, U$10G$16.6
- new net BL-15-2: Q9G$2.D, U$10G$8.6
- new net BL-2-1: U$9G$3.6
- new net BL-2-2: U$9G$11.6
- new net BL-3-1: U$9G$4.6
- new net BL-3-2: U$9G$12.6
- new net BL-4-1: Q4G$1.D, U$10G$11.6
- new net BL-4-2: Q4G$2.D, U$10G$3.6
- new net BL-5-1: Q5G$1.D, U$10G$12.6
- new net BL-5-2: Q5G$2.D, U$10G$4.6
- new net BL-6-1: U$9G$1.6
- new net BL-6-2: U$9G$9.6
- new net BL-7-1: U$9G$2.6
- new net BL-7-2: U$9G$10.6
- new net BL-8-1: Q6G$1.D, U$10G$13.6
- new net BL-8-2: Q6G$2.D, U$10G$5.6
- new net BL-9-1: U$9G$7.6
- new net BL-9-2: U$9G$15.6
- new net DATA-0-1: U$10G$9.1, U$8.4B1
- new net DATA-0-2: U$10G$1.1, U$8.4B2
- new net DATA-1-1: U$10G$10.1, U$8.3B1
- new net DATA-1-2: U$10G$2.1, U$8.3B2
- new net DATA-10-1: U$7.8B1, U$9G$8.1
- new net DATA-10-2: U$7.8B2, U$9G$16.1
- new net DATA-11-1: U$10G$14.1, U$7.11B1
- new net DATA-11-2: U$10G$6.1, U$7.11B2
- new net DATA-12-1: U$7.6B1, U$9G$6.1
- new net DATA-12-2: U$7.6B2, U$9G$14.1
- new net DATA-13-1: U$7.5B1, U$9G$5.1
- new net DATA-13-2: U$7.5B2, U$9G$13.1
- new net DATA-14-1: U$10G$15.1, U$7.10B1
- new net DATA-14-2: U$10G$7.1, U$7.10B2
- new net DATA-15-1: U$10G$16.1, U$7.9B1
- new net DATA-15-2: U$10G$8.1, U$7.9B2
- new net DATA-2-1: U$7.3B1, U$9G$3.1
- new net DATA-2-2: U$7.3B2, U$9G$11.1
- new net DATA-3-1: U$7.4B1, U$9G$4.1
- new net DATA-3-2: U$7.4B2, U$9G$12.1
- new net DATA-4-1: U$10G$11.1, U$8.2B1
- new net DATA-4-2: U$10G$3.1, U$8.2B2
- new net DATA-5-1: U$10G$12.1, U$8.1B1
- new net DATA-5-2: U$10G$4.1, U$8.1B2
- new net DATA-6-1: U$7.1B1, U$9G$1.1
- new net DATA-6-2: U$7.1B2, U$9G$9.1
- new net DATA-7-1: U$7.2B1, U$9G$2.1
- new net DATA-7-2: U$7.2B2, U$9G$10.1
- new net DATA-8-1: U$10G$13.1, U$7.12B1
- new net DATA-8-2: U$10G$5.1, U$7.12B2
- new net DATA-9-1: U$7.7B1, U$9G$7.1
- new net DATA-9-2: U$7.7B2, U$9G$15.1
- new net DC: U$10G$1.4, U$10G$10.4, U$10G$11.4, U$10G$12.4, U$10G$13.4, U$10G$14.4, U$10G$15.4, U$10G$16.4, U$10G$2.4, U$10G$3.4, U$10G$4.4, U$10G$5.4, U$10G$6.4, U$10G$7.4, U$10G$8.4, U$10G$9.4, U$9G$1.4, U$9G$10.4, U$9G$11.4, U$9G$12.4, U$9G$13.4, U$9G$14.4, U$9G$15.4, U$9G$16.4, U$9G$2.4, U$9G$3.4, U$9G$4.4, U$9G$5.4, U$9G$6.4, U$9G$7.4, U$9G$8.4, U$9G$9.4
- new net MUX_S: U$1.GPIO2_24, U$7.S, U$8.S
- new net N$10: Q14G$2.D
- new net N$11: Q15G$1.D
- new net N$12: Q15G$2.D
- new net N$13: Q16G$1.D
- new net N$14: Q16G$2.D
- new net N$15: Q1G$1.D
- new net N$16: Q1G$2.D
- new net N$17: Q10G$1.D
- new net N$18: Q10G$2.D
- new net N$19: Q11G$1.D
- new net N$20: Q11G$2.D
- new net N$21: Q12G$1.D
- new net N$22: U$9G$6.6
- new net N$23: Q12G$2.D
- new net N$5: Q13G$1.D
- new net N$6: Q13G$2.D
- new net N$9: Q14G$1.D
- new net PWM0: Q2G$1.G, U$1.CLKOUT2
- new net PWM1: Q2G$2.G, U$1.GPIO0_7
- new net PWM10: Q7G$1.G, U$1.GPIO1_17
- new net PWM11: Q7G$2.G, U$1.UART2_RXD
- new net PWM12: Q8G$1.G, U$1.UART2_TXD
- new net PWM13: Q8G$2.G, U$1.I2C2_SDA
- new net PWM14: Q9G$1.G, U$1.I2C2_SCL
- new net PWM15: Q9G$2.G, U$1.I2C1_SDA
- new net PWM16: Q1G$1.G, U$1.GPIO2_6
- new net PWM17: Q1G$2.G, U$1.GPIO2_7
- new net PWM18: Q10G$1.G, U$1.GPIO2_8
- new net PWM19: Q10G$2.G, U$1.GPIO2_9
- new net PWM2: Q3G$1.G, U$1.SPI1_SCLK
- new net PWM20: Q11G$1.G, U$1.GPIO2_10
- new net PWM21: Q11G$2.G, U$1.GPIO2_11
- new net PWM22: Q12G$1.G, U$1.GPIO2_12
- new net PWM23: Q12G$2.G, U$1.GPIO2_13
- new net PWM24: Q13G$1.G, U$1.UART5_TXD
- new net PWM25: Q13G$2.G, U$1.UART5_RXD
- new net PWM26: Q14G$1.G, U$1.UART4_CTSN
- new net PWM27: Q14G$2.G, U$1.UART3_CTSN
- new net PWM28: Q15G$1.G, U$1.UART4_RTSN
- new net PWM29: Q15G$2.G, U$1.UART3_RTSN
- new net PWM3: Q3G$2.G, U$1.SPI1_DI
- new net PWM30: Q16G$1.G, U$1.UART5_CTSN
- new net PWM31: Q16G$2.G, U$1.UART5_RTSN
- new net PWM4: Q4G$1.G, U$1.SPI1_DO
- new net PWM5: Q4G$2.G, U$1.SPI1_CS0
- new net PWM6: Q5G$1.G, U$1.GPIO3_19
- new net PWM7: Q5G$2.G, U$1.UART1_RXD
- new net PWM8: Q6G$1.G, U$1.GPIO3_21
- new net PWM9: Q6G$2.G, U$1.UART1_TXD
- new net SCL-A-1: U$8.5B1, U$9G$1.8, U$9G$2.8
- new net SCL-A-2: U$8.5B2, U$9G$10.8, U$9G$9.8
- new net SCL-B-1: U$8.6B1, U$9G$3.8, U$9G$4.8
- new net SCL-B-2: U$8.6B2, U$9G$11.8, U$9G$12.8
- new net SCL-C-1: U$8.7B1, U$9G$5.8, U$9G$6.8
- new net SCL-C-2: U$8.7B2, U$9G$13.8, U$9G$14.8
- new net SCL-D-1: U$8.8B1, U$9G$7.8, U$9G$8.8
- new net SCL-D-2: U$8.8B2, U$9G$15.8, U$9G$16.8
- new net SCL-E-1: U$10G$15.8, U$10G$16.8, U$8.9B1
- new net SCL-E-2: U$10G$7.8, U$10G$8.8, U$8.9B2
- new net SCL-F-1: U$10G$13.8, U$10G$14.8, U$8.10B1
- new net SCL-F-2: U$10G$5.8, U$10G$6.8, U$8.10B2
- new net SCL-G-1: U$10G$11.8, U$10G$12.8, U$8.11B1
- new net SCL-G-2: U$10G$3.8, U$10G$4.8, U$8.11B2
- new net SCL-H-1: U$10G$10.8, U$10G$9.8, U$8.12B1
- new net SCL-H-2: U$10G$1.8, U$10G$2.8, U$8.12B2
- net GND: now also Q10G$1.S, Q10G$2.S, Q11G$1.S, Q11G$2.S, Q12G$1.S, Q12G$2.S, Q13G$1.S, Q13G$2.S, Q14G$1.S, Q14G$2.S, Q15G$1.S, Q15G$2.S, Q16G$1.S, Q16G$2.S, Q1G$1.S, Q1G$2.S, U$10G$1.2, U$10G$1.7, U$10G$10.2, U$10G$10.7, U$10G$11.2, U$10G$11.7, U$10G$12.2, U$10G$12.7, U$10G$13.2, U$10G$13.7, U$10G$14.2, U$10G$14.7, U$10G$15.2, U$10G$15.7, U$10G$16.2, U$10G$16.7, U$10G$2.2, U$10G$2.7, U$10G$3.2, U$10G$3.7, U$10G$4.2, U$10G$4.7, U$10G$5.2, U$10G$5.7, U$10G$6.2, U$10G$6.7, U$10G$7.2, U$10G$7.7, U$10G$8.2, U$10G$8.7, U$10G$9.2, U$10G$9.7, U$9G$1.2, U$9G$1.7, U$9G$10.2, U$9G$10.7, U$9G$11.2, U$9G$11.7, U$9G$12.2, U$9G$12.7, U$9G$13.2, U$9G$13.7, U$9G$14.2, U$9G$14.7, U$9G$15.2, U$9G$15.7, U$9G$16.2, U$9G$16.7, U$9G$2.2, U$9G$2.7, U$9G$3.2, U$9G$3.7, U$9G$4.2, U$9G$4.7, U$9G$5.2, U$9G$5.7, U$9G$6.2, U$9G$6.7, U$9G$7.2, U$9G$7.7, U$9G$8.2, U$9G$8.7, U$9G$9.2, U$9G$9.7; no longer C22.2, C23.2, C7.2, GND.TP, J1.A2, J1.A7, J1.B2, J1.B7, J1.C2, J1.C7, J1.D2, J1.D7, J1.E2, J1.E7, J1.F2, J1.F7, J1.G2, J1.G7, J1.H2, J1.H7, J2.A2, J2.A7, J2.B2, J2.B7, J2.C2, J2.C7, J2.D2, J2.D7, J2.E2, J2.E7, J2.F2, J2.F7, J2.G2, J2.G7, J2.H2, J2.H7
- net RST: now also U$10G$1.5, U$10G$10.5, U$10G$11.5, U$10G$12.5, U$10G$13.5, U$10G$14.5, U$10G$15.5, U$10G$16.5, U$10G$2.5, U$10G$3.5, U$10G$4.5, U$10G$5.5, U$10G$6.5, U$10G$7.5, U$10G$8.5, U$10G$9.5, U$9G$1.5, U$9G$10.5, U$9G$11.5, U$9G$12.5, U$9G$13.5, U$9G$14.5, U$9G$15.5, U$9G$16.5, U$9G$2.5, U$9G$3.5, U$9G$4.5, U$9G$5.5, U$9G$6.5, U$9G$7.5, U$9G$8.5, U$9G$9.5; no longer J1.A5, J1.B5, J1.C5, J1.D5, J1.E5, J1.F5, J1.G5, J1.H5, J2.A5, J2.B5, J2.C5, J2.D5, J2.E5, J2.F5, J2.G5, J2.H5
- net VCC3V3: now also U$10G$1.3, U$10G$10.3, U$10G$11.3, U$10G$12.3, U$10G$13.3, U$10G$14.3, U$10G$15.3, U$10G$16.3, U$10G$2.3, U$10G$3.3, U$10G$4.3, U$10G$5.3, U$10G$6.3, U$10G$7.3, U$10G$8.3, U$10G$9.3, U$9G$1.3, U$9G$10.3, U$9G$11.3, U$9G$12.3, U$9G$13.3, U$9G$14.3, U$9G$15.3, U$9G$16.3, U$9G$2.3, U$9G$3.3, U$9G$4.3, U$9G$5.3, U$9G$6.3, U$9G$7.3, U$9G$8.3, U$9G$9.3; no longer 3V.TP, C22.1, C23.1, C7.1, J1.A3, J1.B3, J1.C3, J1.D3, J1.E3, J1.F3, J1.G3, J1.H3, J2.A3, J2.B3, J2.C3, J2.D3, J2.E3, J2.F3, J2.G3, J2.H3
- net VCC5V: no longer 5V.TP
Other:
- note added: "LOWER"
- note added: "UPPER"
- moved on the sheet: J3

Commit message: More routing
Connections:
- removed net N$10: Q14G$2.D
- removed net N$11: Q15G$1.D
- removed net N$12: Q15G$2.D
- removed net N$13: Q16G$1.D
- removed net N$14: Q16G$2.D
- removed net N$15: Q1G$1.D
- removed net N$16: Q1G$2.D
- removed net N$17: Q10G$1.D
- removed net N$18: Q10G$2.D
- removed net N$19: Q11G$1.D
- removed net N$20: Q11G$2.D
- removed net N$21: Q12G$1.D
- removed net N$22: U$9G$6.6
- removed net N$23: Q12G$2.D
- removed net N$5: Q13G$1.D
- removed net N$6: Q13G$2.D
- removed net N$9: Q14G$1.D
- new net BL-12-1: Q14G$2.D, U$9G$6.6
- net BL-10-1: now also Q16G$2.D
- net BL-10-2: now also Q16G$1.D
- net BL-12-2: now also Q14G$1.D
- net BL-13-1: now also Q12G$2.D
- net BL-13-2: now also Q12G$1.D
- net BL-2-1: now also Q11G$1.D
- net BL-2-2: now also Q11G$2.D
- net BL-3-1: now also Q13G$2.D
- net BL-3-2: now also Q13G$1.D
- net BL-6-1: now also Q1G$1.D
- net BL-6-2: now also Q1G$2.D
- net BL-7-1: now also Q10G$1.D
- net BL-7-2: now also Q10G$2.D
- net BL-9-1: now also Q15G$2.D
- net BL-9-2: now also Q15G$1.D
