File: Hardware/cape.sch (EAGLE design)
At the start: 48 parts, among them IC1 74VHC541, IC2 74VHC541, IC3 74VHC541, IC4 74VHC541, IC5 74VHC541, IC6 74VHC541, IC7 74VHC541, IC8 74VHC541, IC9 74VHC541, J3 RJ45-8P8C, Q1 N-MOSFET-DUALSO8, Q10 N-MOSFET-DUALSO8, Q11 N-MOSFET-DUALSO8, Q12 N-MOSFET-DUALSO8, Q13 N-MOSFET-DUALSO8, Q14 N-MOSFET-DUALSO8, Q15 N-MOSFET-DUALSO8, Q16 N-MOSFET-DUALSO8, Q2 N-MOSFET-DUALSO8, Q3 N-MOSFET-DUALSO8, Q4 N-MOSFET-DUALSO8, Q5 N-MOSFET-DUALSO8, Q6 N-MOSFET-DUALSO8, Q7 N-MOSFET-DUALSO8, Q8 N-MOSFET-DUALSO8, Q9 N-MOSFET-DUALSO8

Commit message: so much routing
Parts:
- removed J3: RJ45-8P8C, cape:RJ45-8P8C
- added J1: MOLEX-P4, cape:MOLEX-P4
- added R8, R9: RESISTOR-X80603, cape:RESISTOR-X80603
Connections:
- removed net 10A: IC1.Y2, IC3.Y2
- removed net 11A: IC1.Y3, IC3.Y3
- removed net 12A: IC1.Y4, IC3.Y4
- removed net 13A: IC1.Y5, IC3.Y5
- removed net 14A: IC1.Y6, IC3.Y6
- removed net 15A: IC1.Y7, IC3.Y7
- removed net 16A: IC1.Y8, IC3.Y8
- removed net 9A: IC1.Y1, IC3.Y1
- removed net SCL-E-1: U$10G$15.8, U$10G$16.8
- removed net SCL-E-2: U$10G$7.8, U$10G$8.8
- removed net SCL-F-1: U$10G$13.8, U$10G$14.8
- removed net SCL-F-2: U$10G$5.8, U$10G$6.8
- removed net SCL-G-1: U$10G$11.8, U$10G$12.8
- removed net SCL-G-2: U$10G$3.8, U$10G$4.8
- removed net SCL-H-1: U$10G$10.8, U$10G$9.8
- removed net SCL-H-2: U$10G$1.8, U$10G$2.8
- new net N$55: IC1.Y1, R8.1A
- new net N$56: IC1.Y2, R8.2A
- new net N$57: IC1.Y3, R8.3A
- new net N$58: IC1.Y4, R8.4A
- new net N$59: IC1.Y5, R8.5A
- new net N$60: IC1.Y6, R8.6A
- new net N$61: IC1.Y7, R8.7A
- new net N$62: IC1.Y8, R8.8A
- new net N$63: IC3.Y1, R9.1A
- new net N$64: IC3.Y2, R9.2A
- new net N$65: IC3.Y3, R9.3A
- new net N$66: IC3.Y4, R9.4A
- new net N$67: IC3.Y5, R9.5A
- new net N$68: IC3.Y6, R9.6A
- new net N$69: IC3.Y7, R9.7A
- new net N$70: IC3.Y8, R9.8A
- new net RST_RAW: IC2.A5, U$1.GPIO1_31
- new net SCL0_A: R9.1B, U$10G$9.8
- new net SCL10_A: R8.1B, U$10G$13.8
- new net SCL11_A: R9.6B, U$10G$3.8
- new net SCL12_A: R8.3B, U$10G$14.8
- new net SCL13_A: R8.4B, U$10G$6.8
- new net SCL14_A: R9.7B, U$10G$12.8
- new net SCL15_A: R9.8B, U$10G$4.8
- new net SCL1_A: R9.2B, U$10G$1.8
- new net SCL2_A: R8.5B, U$10G$15.8
- new net SCL3_A: R8.6B, U$10G$7.8
- new net SCL4_A: R9.3B, U$10G$10.8
- new net SCL5_A: R9.4B, U$10G$2.8
- new net SCL6_A: R8.7B, U$10G$16.8
- new net SCL7_A: R8.8B, U$10G$8.8
- new net SCL8_A: R9.5B, U$10G$11.8
- new net SCL9_A: R8.2B, U$10G$5.8
- net BL-0-1: now also U$10G$1.6; no longer U$10G$9.6
- net BL-0-2: now also U$10G$9.6; no longer U$10G$1.6
- net BL-1-1: now also U$10G$2.6; no longer U$10G$10.6
- net BL-1-2: now also U$10G$10.6; no longer U$10G$2.6
- net BL-10-1: now also U$9G$16.6; no longer U$9G$8.6
- net BL-10-2: now also U$9G$8.6; no longer U$9G$16.6
- net BL-12-1: now also U$9G$14.6; no longer U$9G$6.6
- net BL-12-2: now also U$9G$6.6; no longer U$9G$14.6
- net BL-13-1: now also U$9G$13.6; no longer U$9G$5.6
- net BL-13-2: now also U$9G$5.6; no longer U$9G$13.6
- net BL-3-1: now also U$9G$12.6; no longer U$9G$4.6
- net BL-3-2: now also U$9G$4.6; no longer U$9G$12.6
- net BL-4-1: now also U$10G$3.6; no longer U$10G$11.6
- net BL-4-2: now also U$10G$11.6; no longer U$10G$3.6
- net BL-5-1: now also U$10G$4.6; no longer U$10G$12.6
- net BL-5-2: now also U$10G$12.6; no longer U$10G$4.6
- net BL-9-1: now also U$9G$15.6; no longer U$9G$7.6
- net BL-9-2: now also U$9G$7.6; no longer U$9G$15.6
- net BUF0_A: now also U$10G$4.1; no longer U$10G$9.1
- net BUF10_A: now also U$10G$5.1; no longer U$10G$13.1
- net BUF11_A: now also U$10G$1.1; no longer U$10G$3.1
- net BUF12_A: now also U$10G$16.1; no longer U$10G$14.1
- net BUF13_A: now also U$10G$8.1; no longer U$10G$6.1
- net BUF15_A: now also U$10G$9.1; no longer U$10G$4.1
- net BUF1_A: now also U$10G$3.1; no longer U$10G$1.1
- net BUF2_A: now also U$10G$7.1; no longer U$10G$15.1
- net BUF3_A: now also U$10G$15.1; no longer U$10G$7.1
- net BUF4_A: now also U$10G$11.1; no longer U$10G$10.1
- net BUF6_A: now also U$10G$6.1; no longer U$10G$8.1
- net BUF7_A: now also U$10G$14.1; no longer U$10G$16.1
- net BUF8_A: now also U$10G$10.1; no longer U$10G$11.1
- net BUF9_A: now also U$10G$13.1; no longer U$10G$5.1
- net DC: now also R5.6B
- net DC_RAW: now also IC2.A6
- net GND: now also J1.1, J1.2; no longer IC2.G1, IC4.G1, IC5.G1, IC8.G1, IC9.G1, J3.1, J3.3, J3.5, J3.7
- net MUX_S: now also IC1.G2, IC3.G2, IC6.G2, IC7.G2
- net N$5: now also IC2.Y5, R5.5A; no longer IC2.A5
- net N$6: now also IC2.Y6, R5.6A; no longer IC2.A6
- net PWM16: now also U$1.UART5_RTSN; no longer U$1.GPIO2_6
- net PWM17: now also U$1.UART5_CTSN; no longer U$1.GPIO2_7
- net PWM18: now also U$1.UART3_RTSN; no longer U$1.GPIO2_8
- net PWM19: now also U$1.UART4_RTSN; no longer U$1.GPIO2_9
- net PWM20: now also U$1.UART3_CTSN; no longer U$1.GPIO2_10
- net PWM21: now also U$1.UART4_CTSN; no longer U$1.GPIO2_11
- net PWM22: now also U$1.GPIO2_13; no longer U$1.GPIO2_12
- net PWM23: now also U$1.GPIO2_12; no longer U$1.GPIO2_13
- net PWM24: now also U$1.UART5_RXD; no longer U$1.UART5_TXD
- net PWM25: now also U$1.UART5_TXD; no longer U$1.UART5_RXD
- net PWM26: now also U$1.GPIO2_11; no longer U$1.UART4_CTSN
- net PWM27: now also U$1.GPIO2_10; no longer U$1.UART3_CTSN
- net PWM28: now also U$1.GPIO2_9; no longer U$1.UART4_RTSN
- net PWM29: now also U$1.GPIO2_8; no longer U$1.UART3_RTSN
- net PWM30: now also U$1.GPIO2_7; no longer U$1.UART5_CTSN
- net PWM31: now also U$1.GPIO2_6; no longer U$1.UART5_RTSN
- net RST: now also R5.5B; no longer U$1.GPIO1_31
- net VCC3V3: now also J1.3, J1.4
- net VCC5V: now also IC1.G1, IC2.G1, IC3.G1, IC4.G1, IC5.G1, IC6.G1, IC7.G1, IC8.G1, IC9.G1; no longer J3.2, J3.4, J3.6, J3.8

Commit message: Done routing
Parts:
- added DC_RAW, MUX_S, RST_RAW, SCL_RAW: PTR1TP10R, tenna_avr_AD7021_v0_9_shrink:PTR1TP10R
- added GND: PTR1TP15SQ, tenna_avr_AD7021_v0_9_shrink:PTR1TP15SQ
- added R10, R11, R12, R13, R14, R15, R16, R17, R18, R19, R20, R21, R22, R23, R24, R25, R26, R27, R28, R29, R30, R31, R32, R33: (no value), SparkFun-Passives:RESISTOR0603-RES
- added VCC3V3_TP, VCC5V_TP: PTR1TP15R, tenna_avr_AD7021_v0_9_shrink:PTR1TP15R
- renumbered U$10 to J2, U$9 to J3
Connections:
- removed net N$1: IC2.A1
- removed net N$2: IC2.A2
- removed net N$3: IC2.A3
- removed net N$4: IC2.A4
- net DC_RAW: now also DC_RAW.TP
- net GND: now also GND.TP, R10.2, R11.2, R12.2, R13.2, R14.2, R15.2, R16.2, R17.2, R18.2, R19.2, R20.2, R21.2, R22.2, R23.2, R24.2, R25.2, R26.2, R27.2, R28.2, R29.2, R30.2, R31.2, R32.2, R33.2
- net MUX_S: now also MUX_S.TP
- net PWM0: now also U$1.GPIO0_7; no longer U$1.CLKOUT2
- net PWM1: now also U$1.CLKOUT2; no longer U$1.GPIO0_7
- net PWM10: now also U$1.UART2_TXD; no longer U$1.GPIO1_17
- net PWM11: now also U$1.UART1_TXD; no longer U$1.UART2_RXD
- net PWM12: now also U$1.I2C2_SCL; no longer U$1.UART2_TXD
- net PWM13: now also U$1.UART2_RXD; no longer U$1.I2C2_SDA
- net PWM14: now also U$1.I2C1_SDA; no longer U$1.I2C2_SCL
- net PWM15: now also U$1.I2C2_SDA; no longer U$1.I2C1_SDA
- net PWM2: now also U$1.SPI1_DO; no longer U$1.SPI1_SCLK
- net PWM3: now also U$1.SPI1_SCLK; no longer U$1.SPI1_DI
- net PWM4: now also U$1.GPIO3_19; no longer U$1.SPI1_DO
- net PWM5: now also U$1.SPI1_DI; no longer U$1.SPI1_CS0
- net PWM6: now also U$1.GPIO3_21; no longer U$1.GPIO3_19
- net PWM7: now also U$1.SPI1_CS0; no longer U$1.UART1_RXD
- net PWM8: now also U$1.GPIO1_17; no longer U$1.GPIO3_21
- net PWM9: now also U$1.UART1_RXD; no longer U$1.UART1_TXD
- net RST_RAW: now also RST_RAW.TP
- net SCL0_B: now also R24.1
- net SCL10_A: now also R26.1
- net SCL10_B: now also R16.1
- net SCL11_B: now also R21.1
- net SCL12_A: now also R28.1
- net SCL12_B: now also R14.1
- net SCL13_A: now also R29.1
- net SCL13_B: now also R15.1
- net SCL14_B: now also R19.1
- net SCL15_B: now also R18.1
- net SCL1_B: now also R25.1
- net SCL2_A: now also R30.1
- net SCL2_B: now also R13.1
- net SCL3_A: now also R31.1
- net SCL3_B: now also R12.1
- net SCL4_B: now also R22.1
- net SCL5_B: now also R23.1
- net SCL6_A: now also R32.1
- net SCL6_B: now also R11.1
- net SCL7_A: now also R33.1
- net SCL7_B: now also R10.1
- net SCL8_B: now also R20.1
- net SCL9_A: now also R27.1
- net SCL9_B: now also R17.1
- net SCL_RAW: now also SCL_RAW.TP
- net VCC3V3: now also VCC3V3_TP.TP; no longer U$1.VDD_3V3EXP@2
- net VCC5V: now also VCC5V_TP.TP
Other:
- moved on the sheet: C1, C2, IC1, IC3, R8, R9
