File: Hardware/cape.sch (EAGLE design)
At the start: 81 parts, among them IC1 74VHC541, IC2 74VHC541, IC3 74VHC541, IC4 74VHC541, IC5 74VHC541, IC6 74VHC541, IC7 74VHC541, IC8 74VHC541, IC9 74VHC541, J1 MOLEX-P4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

Commit message: Oops, adding resistors
Parts:
- added R34, R35, R36, R37, R38, R39, R40, R41: (no value), SparkFun-Passives:RESISTOR0603-RES
Connections:
- net GND: now also R34.2, R35.2, R36.2, R37.2, R38.2, R39.2, R40.2, R41.2
- net SCL0_A: now also R34.1
- net SCL11_A: now also R39.1
- net SCL14_A: now also R40.1
- net SCL15_A: now also R41.1
- net SCL1_A: now also R35.1
- net SCL4_A: now also R36.1
- net SCL5_A: now also R37.1
- net SCL8_A: now also R38.1
Changed lines of the file:
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@@
 <part name="GND" library="tenna_avr_AD7021_v0_9_shrink" deviceset="PTR1" device="TP15SQ"/>
 <part name="VCC3V3_TP" library="tenna_avr_AD7021_v0_9_shrink" deviceset="PTR1" device="TP15R"/>
+<part name="R34" library="SparkFun-Passives" deviceset="RESISTOR" device="0603-RES"/>
+<part name="R35" library="SparkFun-Passives" deviceset="RESISTOR" device="0603-RES"/>
+<part name="R36" library="SparkFun-Passives" deviceset="RESISTOR" device="0603-RES"/>
+<part name="R37" library="SparkFun-Passives" deviceset="RESISTOR" device="0603-RES"/>
+<part name="R38" library="SparkFun-Passives" deviceset="RESISTOR" device="0603-RES"/>
+<part name="R39" library="SparkFun-Passives" deviceset="RESISTOR" device="0603-RES"/>
+<part name="R40" library="SparkFun-Passives" deviceset="RESISTOR" device="0603-RES"/>
+<part name="R41" library="SparkFun-Passives" deviceset="RESISTOR" device="0603-RES"/>
+<part name="GND65" library="SparkFun-Aesthetics" deviceset="GND" device=""/>
 </parts>
 <sheets>
@@
 <instance part="GND" gate="G$1" x="287.02" y="20.32"/>
 <instance part="VCC3V3_TP" gate="G$1" x="276.86" y="20.32"/>
+<instance part="R34" gate="G$1" x="20.32" y="-91.44"/>
+<instance part="R35" gate="G$1" x="20.32" y="-93.98"/>
+<instance part="R36" gate="G$1" x="20.32" y="-96.52"/>
+<instance part="R37" gate="G$1" x="20.32" y="-99.06"/>
+<instance part="R38" gate="G$1" x="20.32" y="-101.6"/>
+<instance part="R39" gate="G$1" x="20.32" y="-104.14"/>
+<instance part="R40" gate="G$1" x="20.32" y="-106.68"/>
+<instance part="R41" gate="G$1" x="20.32" y="-109.22"/>
+<instance part="GND65" gate="1" x="27.94" y="-114.3"/>
 </instances>
 <busses>
@@
 <label x="287.02" y="25.4" size="1.4224" layer="95" rot="R90" xref="yes"/>
 </segment>
+<segment>
+<pinref part="R34" gate="G$1" pin="2"/>
+<pinref part="GND65" gate="1" pin="GND"/>
+<wire x1="25.4" y1="-91.44" x2="27.94" y2="-91.44" width="0.1524" layer="91"/>
+<wire x1="27.94" y1="-91.44" x2="27.94" y2="-93.98" width="0.1524" layer="91"/>
+<pinref part="R41" gate="G$1" pin="2"/>
+<wire x1="27.94" y1="-93.98" x2="27.94" y2="-96.52" width="0.1524" layer="91"/>
+<wire x1="27.94" y1="-96.52" x2="27.94" y2="-99.06" width="0.1524" layer="91"/>
+<wire x1="27.94" y1="-99.06" x2="27.94" y2="-101.6" width="0.1524" layer="91"/>
+<wire x1="27.94" y1="-101.6" x2="27.94" y2="-104.14" width="0.1524" layer="91"/>
+<wire x1="27.94" y1="-104.14" x2="27.94" y2="-106.68" width="0.1524" layer="91"/>
+<wire x1="27.94" y1="-106.68" x2="27.94" y2="-109.22" width="0.1524" layer="91"/>
+<wire x1="27.94" y1="-109.22" x2="27.94" y2="-111.76" width="0.1524" layer="91"/>
+<wire x1="25.4" y1="-109.22" x2="27.94" y2="-109.22" width="0.1524" layer="91"/>
+<junction x="27.94" y="-109.22"/>
+<pinref part="R40" gate="G$1" pin="2"/>
+<wire x1="25.4" y1="-106.68" x2="27.94" y2="-106.68" width="0.1524" layer="91"/>
+<junction x="27.94" y="-106.68"/>
+<pinref part="R39" gate="G$1" pin="2"/>
+<wire x1="25.4" y1="-104.14" x2="27.94" y2="-104.14" width="0.1524" layer="91"/>
+<junction x="27.94" y="-104.14"/>
+<pinref part="R38" gate="G$1" pin="2"/>
+<wire x1="25.4" y1="-101.6" x2="27.94" y2="-101.6" width="0.1524" layer="91"/>
+<junction x="27.94" y="-101.6"/>
+<pinref part="R37" gate="G$1" pin="2"/>
+<wire x1="25.4" y1="-99.06" x2="27.94" y2="-99.06" width="0.1524" layer="91"/>
+<junction x="27.94" y="-99.06"/>
+<pinref part="R36" gate="G$1" pin="2"/>
+<wire x1="25.4" y1="-96.52" x2="27.94" y2="-96.52" width="0.1524" layer="91"/>
+<junction x="27.94" y="-96.52"/>
+<pinref part="R35" gate="G$1" pin="2"/>
+<wire x1="25.4" y1="-93.98" x2="27.94" y2="-93.98" width="0.1524" layer="91"/>
+<junction x="27.94" y="-93.98"/>
+</segment>
 </net>
 <net name="RST" class="0">
@@
 <label x="-15.24" y="-101.6" size="1.4224" layer="95" xref="yes"/>
 </segment>
+<segment>
+<pinref part="R38" gate="G$1" pin="1"/>
+<wire x1="15.24" y1="-101.6" x2="12.7" y2="-101.6" width="0.1524" layer="91"/>
+<label x="12.7" y="-101.6" size="1.4224" layer="95" rot="R180" xref="yes"/>
+</segment>
 </net>
 <net name="SCL11_A" class="0">
@@
 <label x="-15.24" y="-104.14" size="1.4224" layer="95" xref="yes"/>
 </segment>
+<segment>
+<pinref part="R39" gate="G$1" pin="1"/>
+<wire x1="15.24" y1="-104.14" x2="12.7" y2="-104.14" width="0.1524" layer="91"/>
+<label x="12.7" y="-104.14" size="1.4224" layer="95" rot="R180" xref="yes"/>
+</segment>
 </net>
 <net name="SCL0_A" class="0">
@@
 <label x="-15.24" y="-91.44" size="1.4224" layer="95" xref="yes"/>
 </segment>
+<segment>
+<pinref part="R34" gate="G$1" pin="1"/>
+<wire x1="15.24" y1="-91.44" x2="12.7" y2="-91.44" width="0.1524" layer="91"/>
+<label x="12.7" y="-91.44" size="1.4224" layer="95" rot="R180" xref="yes"/>
+</segment>
 </net>
 <net name="SCL1_A" class="0">
@@
 <label x="-15.24" y="-93.98" size="1.4224" layer="95" xref="yes"/>
 </segment>
+<segment>
+<pinref part="R35" gate="G$1" pin="1"/>
+<wire x1="15.24" y1="-93.98" x2="12.7" y2="-93.98" width="0.1524" layer="91"/>
+<label x="12.7" y="-93.98" size="1.4224" layer="95" rot="R180" xref="yes"/>
+</segment>
 </net>
 <net name="BL-1-2" class="0">
@@
 <label x="-15.24" y="-109.22" size="1.4224" layer="95" xref="yes"/>
 </segment>
+<segment>
+<pinref part="R41" gate="G$1" pin="1"/>
+<wire x1="15.24" y1="-109.22" x2="12.7" y2="-109.22" width="0.1524" layer="91"/>
+<label x="12.7" y="-109.22" size="1.4224" layer="95" rot="R180" xref="yes"/>
+</segment>
 </net>
 <net name="SCL14_A" class="0">
@@
 <label x="-15.24" y="-106.68" size="1.4224" layer="95" xref="yes"/>
 </segment>
+<segment>
+<pinref part="R40" gate="G$1" pin="1"/>
+<wire x1="15.24" y1="-106.68" x2="12.7" y2="-106.68" width="0.1524" layer="91"/>
+<label x="12.7" y="-106.68" size="1.4224" layer="95" rot="R180" xref="yes"/>
+</segment>
 </net>
 <net name="SCL5_A" class="0">
@@
 <label x="-15.24" y="-99.06" size="1.4224" layer="95" xref="yes"/>
 </segment>
+<segment>
+<pinref part="R37" gate="G$1" pin="1"/>
+<wire x1="15.24" y1="-99.06" x2="12.7" y2="-99.06" width="0.1524" layer="91"/>
+<label x="12.7" y="-99.06" size="1.4224" layer="95" rot="R180" xref="yes"/>
+</segment>
 </net>
 <net name="SCL4_A" class="0">
@@
 <label x="-15.24" y="-96.52" size="1.4224" layer="95" xref="yes"/>
 </segment>
+<segment>
+<pinref part="R36" gate="G$1" pin="1"/>
+<wire x1="15.24" y1="-96.52" x2="12.7" y2="-96.52" width="0.1524" layer="91"/>
+<label x="12.7" y="-96.52" size="1.4224" layer="95" rot="R180" xref="yes"/>
+</segment>
 </net>

Commit message: Updating bom info
Parts:
- IC1, IC2, IC3, IC4, IC5, IC6, IC7, IC8, IC9: PARTNO (none) -> MC74LCX245DTR2G
- J2, J3: PARTNO (none) -> 10118074-500A010LF
- Q1, Q10, Q11, Q12, Q13, Q14, Q15, Q16, Q2, Q3, Q4, Q5, Q6, Q7, Q8, Q9: PARTNO * -> DMN6040SSD-13
- R1, R2, R3, R4, R5, R6, R7, R8, R9: PARTNO (none) -> 742C163220JP
