File: Hardware/cape.brd (EAGLE design)
At the start: 128 x 126 mm, 51 parts, among them IC1 74VHC541, IC2 74VHC541, IC3 74VHC541, IC4 74VHC541, IC5 74VHC541, IC6 74VHC541, IC7 74VHC541, IC8 74VHC541, IC9 74VHC541, J3 RJ45-8P8C, Q1 N-MOSFET-DUALSO8, Q10 N-MOSFET-DUALSO8, Q11 N-MOSFET-DUALSO8, Q12 N-MOSFET-DUALSO8, Q13 N-MOSFET-DUALSO8, Q14 N-MOSFET-DUALSO8, Q15 N-MOSFET-DUALSO8, Q16 N-MOSFET-DUALSO8, Q2 N-MOSFET-DUALSO8, Q3 N-MOSFET-DUALSO8, Q4 N-MOSFET-DUALSO8, Q5 N-MOSFET-DUALSO8, Q6 N-MOSFET-DUALSO8, Q7 N-MOSFET-DUALSO8, Q8 N-MOSFET-DUALSO8, Q9 N-MOSFET-DUALSO8

Commit message: so much routing
Parts:
- removed J3: RJ45-8P8C, cape:54602-908LF
- added J1: MOLEX-P4, cape:MOLEX-P4
- added R8, R9: RESISTOR-X80603, cape:R0603-X8
- moved Q16 221.0 mm to (113.2, 3.50), flipped to the bottom
- moved Q15 203.0 mm to (100.0, 3.50), flipped to the bottom
- moved Q14 184.0 mm to (85.6, 3.50), flipped to the bottom
- moved Q12 158.6 mm to (71.7, 3.50), flipped to the bottom
- moved Q13 152.4 mm to (58.2, 3.50), flipped to the bottom
- moved Q11 150.0 mm to (44.1, 3.50), flipped to the bottom
- moved Q10 132.8 mm to (30.6, 3.50), flipped to the bottom
- moved Q2 129.6 mm to (112.0, 129.6), flipped to the bottom
- moved Q3 121.8 mm to (98.6, 129.8), flipped to the bottom
- moved Q1 116.3 mm to (17.0, 3.50), flipped to the bottom
- moved Q4 113.3 mm to (84.8, 128.0), flipped to the bottom
- moved U$12 112.5 mm to (111.0, 51.8)
- moved Q5 104.5 mm to (70.5, 128.0), flipped to the bottom
- moved Q6 97.1 mm to (57.5, 128.0), flipped to the bottom
- moved Q7 88.4 mm to (43.4, 128.0), flipped to the bottom
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Connections:
- removed net 10A: IC1.17, IC3.17
- removed net 11A: IC1.16, IC3.16
- removed net 12A: IC1.15, IC3.15
- removed net 13A: IC1.14, IC3.14
- removed net 14A: IC1.13, IC3.13
- removed net 15A: IC1.12, IC3.12
- removed net 16A: IC1.11, IC3.11
- removed net 9A: IC1.18, IC3.18
- removed net SCL-E-1: U$10.UG8, U$10.UH8
- removed net SCL-E-2: U$10.LG8, U$10.LH8
- removed net SCL-F-1: U$10.UE8, U$10.UF8
- removed net SCL-F-2: U$10.LE8, U$10.LF8
- removed net SCL-G-1: U$10.UC8, U$10.UD8
- removed net SCL-G-2: U$10.LC8, U$10.LD8
- removed net SCL-H-1: U$10.UA8, U$10.UB8
- removed net SCL-H-2: U$10.LA8, U$10.LB8
- new net N$55: IC1.18, R8.1B
- new net N$56: IC1.17, R8.2B
- new net N$57: IC1.16, R8.3B
- new net N$58: IC1.15, R8.4B
- new net N$59: IC1.14, R8.5B
- new net N$60: IC1.13, R8.6B
- new net N$61: IC1.12, R8.7B
- new net N$62: IC1.11, R8.8B
- new net N$63: IC3.18, R9.1B
- new net N$64: IC3.17, R9.2B
- new net N$65: IC3.16, R9.3B
- new net N$66: IC3.15, R9.4B
- new net N$67: IC3.14, R9.5B
- new net N$68: IC3.13, R9.6B
- new net N$69: IC3.12, R9.7B
- new net N$70: IC3.11, R9.8B
- new net RST_RAW: IC2.6, U$1.20
- new net SCL0_A: R9.1A, U$10.UA8
- new net SCL10_A: R8.1A, U$10.UE8
- new net SCL11_A: R9.6A, U$10.LC8
- new net SCL12_A: R8.3A, U$10.UF8
- new net SCL13_A: R8.4A, U$10.LF8
- new net SCL14_A: R9.7A, U$10.UD8
- new net SCL15_A: R9.8A, U$10.LD8
- new net SCL1_A: R9.2A, U$10.LA8
- new net SCL2_A: R8.5A, U$10.UG8
- new net SCL3_A: R8.6A, U$10.LG8
- new net SCL4_A: R9.3A, U$10.UB8
- new net SCL5_A: R9.4A, U$10.LB8
- new net SCL6_A: R8.7A, U$10.UH8
- new net SCL7_A: R8.8A, U$10.LH8
- new net SCL8_A: R9.5A, U$10.UC8
- new net SCL9_A: R8.2A, U$10.LE8
- net BL-0-1: now also U$10.LA6; no longer U$10.UA6
- net BL-0-2: now also U$10.UA6; no longer U$10.LA6
- net BL-1-1: now also U$10.LB6; no longer U$10.UB6
- net BL-1-2: now also U$10.UB6; no longer U$10.LB6
- net BL-10-1: now also U$9.UH6; no longer U$9.LH6
- net BL-10-2: now also U$9.LH6; no longer U$9.UH6
- net BL-12-1: now also U$9.UF6; no longer U$9.LF6
- net BL-12-2: now also U$9.LF6; no longer U$9.UF6
- net BL-13-1: now also U$9.UE6; no longer U$9.LE6
- net BL-13-2: now also U$9.LE6; no longer U$9.UE6
- net BL-3-1: now also U$9.UD6; no longer U$9.LD6
- net BL-3-2: now also U$9.LD6; no longer U$9.UD6
- net BL-4-1: now also U$10.LC6; no longer U$10.UC6
- net BL-4-2: now also U$10.UC6; no longer U$10.LC6
- net BL-5-1: now also U$10.LD6; no longer U$10.UD6
- net BL-5-2: now also U$10.UD6; no longer U$10.LD6
- net BL-9-1: now also U$9.UG6; no longer U$9.LG6
- net BL-9-2: now also U$9.LG6; no longer U$9.UG6
- net BUF0_A: now also U$10.LD1; no longer U$10.UA1
- net BUF10_A: now also U$10.LE1; no longer U$10.UE1
- net BUF11_A: now also U$10.LA1; no longer U$10.LC1
- net BUF12_A: now also U$10.UH1; no longer U$10.UF1
- net BUF13_A: now also U$10.LH1; no longer U$10.LF1
- net BUF15_A: now also U$10.UA1; no longer U$10.LD1
- net BUF1_A: now also U$10.LC1; no longer U$10.LA1
- net BUF2_A: now also U$10.LG1; no longer U$10.UG1
- net BUF3_A: now also U$10.UG1; no longer U$10.LG1
- net BUF4_A: now also U$10.UC1; no longer U$10.UB1
- net BUF6_A: now also U$10.LF1; no longer U$10.LH1
- net BUF7_A: now also U$10.UF1; no longer U$10.UH1
- net BUF8_A: now also U$10.UB1; no longer U$10.UC1
- net BUF9_A: now also U$10.UE1; no longer U$10.LE1
- net DC: now also R5.6A
- net DC_RAW: now also IC2.7
- net GND: now also J1.1, J1.2; no longer IC2.1, IC4.1, IC5.1, IC8.1, IC9.1, J3.2, J3.4, J3.6, J3.8
- net MUX_S: now also IC1.19, IC3.19, IC6.19, IC7.19
- net N$5: now also IC2.14, R5.5B; no longer IC2.6
- net N$6: now also IC2.13, R5.6B; no longer IC2.7
- net PWM16: now also U$1.32; no longer U$1.45
- net PWM17: now also U$1.31; no longer U$1.46
- net PWM18: now also U$1.34; no longer U$1.43
- net PWM19: now also U$1.33; no longer U$1.44
- net PWM20: now also U$1.36; no longer U$1.41
- net PWM21: now also U$1.35; no longer U$1.42
- net PWM22: now also U$1.40; no longer U$1.39
- net PWM23: now also U$1.39; no longer U$1.40
- net PWM24: now also U$1.38; no longer U$1.37
- net PWM25: now also U$1.37; no longer U$1.38
- net PWM26: now also U$1.42; no longer U$1.35
- net PWM27: now also U$1.41; no longer U$1.36
- net PWM28: now also U$1.44; no longer U$1.33
- net PWM29: now also U$1.43; no longer U$1.34
- net PWM30: now also U$1.46; no longer U$1.31
- net PWM31: now also U$1.45; no longer U$1.32
- net RST: now also R5.5A; no longer U$1.20
- net VCC3V3: now also J1.3, J1.4
- net VCC5V: now also IC1.1, IC2.1, IC3.1, IC4.1, IC5.1, IC6.1, IC7.1, IC8.1, IC9.1; no longer J3.1, J3.3, J3.5, J3.7
Routing:
- net DC: track 0.00 -> 754.8 mm, vias 0 -> 8
- net VCC3V3: track 0.00 -> 739.4 mm, vias 0 -> 38
- net RST: track 0.00 -> 737.8 mm, vias 0 -> 24
- net VCC5V: track 0.00 -> 294.2 mm, vias 0 -> 8
- net PWM17: track 0.00 -> 228.8 mm
- net PWM16: track 0.00 -> 227.6 mm
- net PWM19: track 0.00 -> 210.7 mm
- net PWM18: track 0.00 -> 208.8 mm
- net PWM21: track 0.00 -> 191.0 mm
- net PWM20: track 0.00 -> 188.8 mm
- net PWM25: track 0.00 -> 169.8 mm
- net PWM24: track 0.00 -> 168.7 mm
- net BUF4_A: track 0.00 -> 164.9 mm
- net BUF0_A: track 0.00 -> 158.3 mm
- net PWM23: track 0.00 -> 151.5 mm
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Other:
- board size 128 x 126 mm -> 132 x 144 mm
