File: Hardware/cape.brd (EAGLE design)
At the start: 132 x 144 mm, 53 parts, among them IC1 74VHC541, IC2 74VHC541, IC3 74VHC541, IC4 74VHC541, IC5 74VHC541, IC6 74VHC541, IC7 74VHC541, IC8 74VHC541, IC9 74VHC541, J1 MOLEX-P4, Q1 N-MOSFET-DUALSO8, Q10 N-MOSFET-DUALSO8, Q11 N-MOSFET-DUALSO8, Q12 N-MOSFET-DUALSO8, Q13 N-MOSFET-DUALSO8, Q14 N-MOSFET-DUALSO8, Q15 N-MOSFET-DUALSO8, Q16 N-MOSFET-DUALSO8, Q2 N-MOSFET-DUALSO8, Q3 N-MOSFET-DUALSO8, Q4 N-MOSFET-DUALSO8, Q5 N-MOSFET-DUALSO8, Q6 N-MOSFET-DUALSO8, Q7 N-MOSFET-DUALSO8, Q8 N-MOSFET-DUALSO8, Q9 N-MOSFET-DUALSO8

Commit message: Done routing
Parts:
- removed U$10, U$9: RJ45-8P8C-16FCI-16, cape:FCI-10118074-500A010LF
- added DC_RAW, MUX_S, RST_RAW, SCL_RAW: PTR1TP10R, tenna_avr_AD7021_v0_9_shrink:TP10R
- added GND: PTR1TP15SQ, tenna_avr_AD7021_v0_9_shrink:TP15SQ
- added J2, J3: RJ45-8P8C-16FCI-16, cape:FCI-10118074-500A010LF
- added R10, R11, R12, R13, R14, R15, R16, R17, R18, R19, R20, R21, R22, R23, R24, R25, R26, R27, R28, R29, R30, R31, R32, R33: (no value), SparkFun-Passives:0603-RES
- added VCC3V3_TP, VCC5V_TP: PTR1TP15R, tenna_avr_AD7021_v0_9_shrink:TP15R
- moved U$4 165.8 mm to (126.0, 3.00), flipped to the bottom
- moved U$6 29.8 mm to (130.0, 142.0), flipped to the bottom
- moved U$3 19.8 mm to (122.0, 91.5)
- moved U$5 18.7 mm to (8.00, 3.00), flipped to the bottom
- moved U$12 14.7 mm to (122.0, 61.5)
- moved C2 10.0 mm to (74.8, 92.0), turned to 180 degrees
- moved C1 7.00 mm to (43.0, 89.0)
- moved C20 7.00 mm to (36.9, 64.0)
- moved C21 7.00 mm to (50.0, 64.0)
- moved C3 7.00 mm to (65.2, 40.8)
- moved C4 7.00 mm to (76.2, 41.7)
- moved C5 7.00 mm to (25.8, 45.5)
- moved C6 7.00 mm to (59.9, 64.0)
- moved C7 7.00 mm to (40.9, 45.5)
- moved IC1 7.00 mm to (38.0, 89.0)
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Connections:
- removed net N$1: IC2.2
- removed net N$2: IC2.3
- removed net N$3: IC2.4
- removed net N$4: IC2.5
- net BL-0-1: now also J2.LA6; no longer U$10.LA6
- net BL-0-2: now also J2.UA6; no longer U$10.UA6
- net BL-1-1: now also J2.LB6; no longer U$10.LB6
- net BL-1-2: now also J2.UB6; no longer U$10.UB6
- net BL-10-1: now also J3.UH6; no longer U$9.UH6
- net BL-10-2: now also J3.LH6; no longer U$9.LH6
- net BL-11-1: now also J2.UF6; no longer U$10.UF6
- net BL-11-2: now also J2.LF6; no longer U$10.LF6
- net BL-12-1: now also J3.UF6; no longer U$9.UF6
- net BL-12-2: now also J3.LF6; no longer U$9.LF6
- net BL-13-1: now also J3.UE6; no longer U$9.UE6
- net BL-13-2: now also J3.LE6; no longer U$9.LE6
- net BL-14-1: now also J2.UG6; no longer U$10.UG6
- net BL-14-2: now also J2.LG6; no longer U$10.LG6
- net BL-15-1: now also J2.UH6; no longer U$10.UH6
- net BL-15-2: now also J2.LH6; no longer U$10.LH6
- net BL-2-1: now also J3.LC6; no longer U$9.LC6
- net BL-2-2: now also J3.UC6; no longer U$9.UC6
- net BL-3-1: now also J3.UD6; no longer U$9.UD6
- net BL-3-2: now also J3.LD6; no longer U$9.LD6
- net BL-4-1: now also J2.LC6; no longer U$10.LC6
- net BL-4-2: now also J2.UC6; no longer U$10.UC6
- net BL-5-1: now also J2.LD6; no longer U$10.LD6
- net BL-5-2: now also J2.UD6; no longer U$10.UD6
- net BL-6-1: now also J3.LA6; no longer U$9.LA6
- net BL-6-2: now also J3.UA6; no longer U$9.UA6
- net BL-7-1: now also J3.LB6; no longer U$9.LB6
- net BL-7-2: now also J3.UB6; no longer U$9.UB6
- net BL-8-1: now also J2.UE6; no longer U$10.UE6
- net BL-8-2: now also J2.LE6; no longer U$10.LE6
- net BL-9-1: now also J3.UG6; no longer U$9.UG6
- net BL-9-2: now also J3.LG6; no longer U$9.LG6
- net BUF0_A: now also J2.LD1; no longer U$10.LD1
- net BUF0_B: now also J3.LE1; no longer U$9.LE1
- net BUF10_A: now also J2.LE1; no longer U$10.LE1
- net BUF10_B: now also J3.LA1; no longer U$9.LA1
- net BUF11_A: now also J2.LA1; no longer U$10.LA1
- net BUF11_B: now also J3.UG1; no longer U$9.UG1
- net BUF12_A: now also J2.UH1; no longer U$10.UH1
- net BUF12_B: now also J3.LB1; no longer U$9.LB1
- net BUF13_A: now also J2.LH1; no longer U$10.LH1
- net BUF13_B: now also J3.UB1; no longer U$9.UB1
- net BUF14_A: now also J2.UD1; no longer U$10.UD1
- net BUF14_B: now also J3.UH1; no longer U$9.UH1
- net BUF15_A: now also J2.UA1; no longer U$10.UA1
- net BUF15_B: now also J3.LH1; no longer U$9.LH1
- net BUF1_A: now also J2.LC1; no longer U$10.LC1
- net BUF1_B: now also J3.UE1; no longer U$9.UE1
- net BUF2_A: now also J2.LG1; no longer U$10.LG1
- net BUF2_B: now also J3.UC1; no longer U$9.UC1
- net BUF3_A: now also J2.UG1; no longer U$10.UG1
- net BUF3_B: now also J3.LC1; no longer U$9.LC1
- net BUF4_A: now also J2.UC1; no longer U$10.UC1
- net BUF4_B: now also J3.LF1; no longer U$9.LF1
- net BUF5_A: now also J2.LB1; no longer U$10.LB1
- net BUF5_B: now also J3.UF1; no longer U$9.UF1
- net BUF6_A: now also J2.LF1; no longer U$10.LF1
- net BUF6_B: now also J3.UD1; no longer U$9.UD1
- net BUF7_A: now also J2.UF1; no longer U$10.UF1
- net BUF7_B: now also J3.LD1; no longer U$9.LD1
- net BUF8_A: now also J2.UB1; no longer U$10.UB1
- net BUF8_B: now also J3.LG1; no longer U$9.LG1
- net BUF9_A: now also J2.UE1; no longer U$10.UE1
- net BUF9_B: now also J3.UA1; no longer U$9.UA1
- net DC: now also J2.LA4, J2.LB4, J2.LC4, J2.LD4, J2.LE4, J2.LF4, J2.LG4, J2.LH4, J2.UA4, J2.UB4, J2.UC4, J2.UD4, J2.UE4, J2.UF4, J2.UG4, J2.UH4, J3.LA4, J3.LB4, J3.LC4, J3.LD4, J3.LE4, J3.LF4, J3.LG4, J3.LH4, J3.UA4, J3.UB4, J3.UC4, J3.UD4, J3.UE4, J3.UF4, J3.UG4, J3.UH4; no longer U$10.LA4, U$10.LB4, U$10.LC4, U$10.LD4, U$10.LE4, U$10.LF4, U$10.LG4, U$10.LH4, U$10.UA4, U$10.UB4, U$10.UC4, U$10.UD4, U$10.UE4, U$10.UF4, U$10.UG4, U$10.UH4, U$9.LA4, U$9.LB4, U$9.LC4, U$9.LD4, U$9.LE4, U$9.LF4, U$9.LG4, U$9.LH4, U$9.UA4, U$9.UB4, U$9.UC4, U$9.UD4, U$9.UE4, U$9.UF4, U$9.UG4, U$9.UH4
- net DC_RAW: now also DC_RAW.TP
- net GND: now also GND.TP, J2.LA2, J2.LA7, J2.LB2, J2.LB7, J2.LC2, J2.LC7, J2.LD2, J2.LD7, J2.LE2, J2.LE7, J2.LF2, J2.LF7, J2.LG2, J2.LG7, J2.LH2, J2.LH7, J2.UA2, J2.UA7, J2.UB2, J2.UB7, J2.UC2, J2.UC7, J2.UD2, J2.UD7, J2.UE2, J2.UE7, J2.UF2, J2.UF7, J2.UG2, J2.UG7, J2.UH2, J2.UH7, J3.LA2, J3.LA7, J3.LB2, J3.LB7, J3.LC2, J3.LC7, J3.LD2, J3.LD7, J3.LE2, J3.LE7, J3.LF2, J3.LF7, J3.LG2, J3.LG7, J3.LH2, J3.LH7, J3.UA2, J3.UA7, J3.UB2, J3.UB7, J3.UC2, J3.UC7, J3.UD2, J3.UD7, J3.UE2, J3.UE7, J3.UF2, J3.UF7, J3.UG2, J3.UG7, J3.UH2, J3.UH7, R10.2, R11.2, R12.2, R13.2, R14.2, R15.2, R16.2, R17.2, R18.2, R19.2, R20.2, R21.2, R22.2, R23.2, R24.2, R25.2, R26.2, R27.2, R28.2, R29.2, R30.2, R31.2, R32.2, R33.2; no longer U$10.LA2, U$10.LA7, U$10.LB2, U$10.LB7, U$10.LC2, U$10.LC7, U$10.LD2, U$10.LD7, U$10.LE2, U$10.LE7, U$10.LF2, U$10.LF7, U$10.LG2, U$10.LG7, U$10.LH2, U$10.LH7, U$10.UA2, U$10.UA7, U$10.UB2, U$10.UB7, U$10.UC2, U$10.UC7, U$10.UD2, U$10.UD7, U$10.UE2, U$10.UE7, U$10.UF2, U$10.UF7, U$10.UG2, U$10.UG7, U$10.UH2, U$10.UH7, U$9.LA2, U$9.LA7, U$9.LB2, U$9.LB7, U$9.LC2, U$9.LC7, U$9.LD2, U$9.LD7, U$9.LE2, U$9.LE7, U$9.LF2, U$9.LF7, U$9.LG2, U$9.LG7, U$9.LH2, U$9.LH7, U$9.UA2, U$9.UA7, U$9.UB2, U$9.UB7, U$9.UC2, U$9.UC7, U$9.UD2, U$9.UD7, U$9.UE2, U$9.UE7, U$9.UF2, U$9.UF7, U$9.UG2, U$9.UG7, U$9.UH2, U$9.UH7
- net MUX_S: now also MUX_S.TP
- net PWM0: now also U$1.88; no longer U$1.87
- net PWM1: now also U$1.87; no longer U$1.88
- net PWM10: now also U$1.67; no longer U$1.69
- net PWM11: now also U$1.70; no longer U$1.68
- net PWM12: now also U$1.65; no longer U$1.67
- net PWM13: now also U$1.68; no longer U$1.66
- net PWM14: now also U$1.64; no longer U$1.65
- net PWM15: now also U$1.66; no longer U$1.64
- net PWM2: now also U$1.75; no longer U$1.77
- net PWM3: now also U$1.77; no longer U$1.76
- net PWM4: now also U$1.73; no longer U$1.75
- net PWM5: now also U$1.76; no longer U$1.74
- net PWM6: now also U$1.71; no longer U$1.73
- net PWM7: now also U$1.74; no longer U$1.72
- net PWM8: now also U$1.69; no longer U$1.71
- net PWM9: now also U$1.72; no longer U$1.70
- net RST: now also J2.LA5, J2.LB5, J2.LC5, J2.LD5, J2.LE5, J2.LF5, J2.LG5, J2.LH5, J2.UA5, J2.UB5, J2.UC5, J2.UD5, J2.UE5, J2.UF5, J2.UG5, J2.UH5, J3.LA5, J3.LB5, J3.LC5, J3.LD5, J3.LE5, J3.LF5, J3.LG5, J3.LH5, J3.UA5, J3.UB5, J3.UC5, J3.UD5, J3.UE5, J3.UF5, J3.UG5, J3.UH5; no longer U$10.LA5, U$10.LB5, U$10.LC5, U$10.LD5, U$10.LE5, U$10.LF5, U$10.LG5, U$10.LH5, U$10.UA5, U$10.UB5, U$10.UC5, U$10.UD5, U$10.UE5, U$10.UF5, U$10.UG5, U$10.UH5, U$9.LA5, U$9.LB5, U$9.LC5, U$9.LD5, U$9.LE5, U$9.LF5, U$9.LG5, U$9.LH5, U$9.UA5, U$9.UB5, U$9.UC5, U$9.UD5, U$9.UE5, U$9.UF5, U$9.UG5, U$9.UH5
- net RST_RAW: now also RST_RAW.TP
- net SCL0_A: now also J2.UA8; no longer U$10.UA8
- net SCL0_B: now also J3.UH8, R24.1; no longer U$9.UH8
- net SCL10_A: now also J2.UE8, R26.1; no longer U$10.UE8
- net SCL10_B: now also J3.UD8, R16.1; no longer U$9.UD8
- net SCL11_A: now also J2.LC8; no longer U$10.LC8
- net SCL11_B: now also J3.LF8, R21.1; no longer U$9.LF8
- net SCL12_A: now also J2.UF8, R28.1; no longer U$10.UF8
- net SCL12_B: now also J3.UC8, R14.1; no longer U$9.UC8
- net SCL13_A: now also J2.LF8, R29.1; no longer U$10.LF8
- net SCL13_B: now also J3.LC8, R15.1; no longer U$9.LC8
- net SCL14_A: now also J2.UD8; no longer U$10.UD8
- net SCL14_B: now also J3.LE8, R19.1; no longer U$9.LE8
- net SCL15_A: now also J2.LD8; no longer U$10.LD8
- net SCL15_B: now also J3.UE8, R18.1; no longer U$9.UE8
- net SCL1_A: now also J2.LA8; no longer U$10.LA8
- net SCL1_B: now also J3.LH8, R25.1; no longer U$9.LH8
- net SCL2_A: now also J2.UG8, R30.1; no longer U$10.UG8
- net SCL2_B: now also J3.LB8, R13.1; no longer U$9.LB8
- net SCL3_A: now also J2.LG8, R31.1; no longer U$10.LG8
- net SCL3_B: now also J3.UB8, R12.1; no longer U$9.UB8
- net SCL4_A: now also J2.UB8; no longer U$10.UB8
- net SCL4_B: now also J3.UG8, R22.1; no longer U$9.UG8
- net SCL5_A: now also J2.LB8; no longer U$10.LB8
- net SCL5_B: now also J3.LG8, R23.1; no longer U$9.LG8
- net SCL6_A: now also J2.UH8, R32.1; no longer U$10.UH8
- net SCL6_B: now also J3.LA8, R11.1; no longer U$9.LA8
- net SCL7_A: now also J2.LH8, R33.1; no longer U$10.LH8
- net SCL7_B: now also J3.UA8, R10.1; no longer U$9.UA8
- net SCL8_A: now also J2.UC8; no longer U$10.UC8
- net SCL8_B: now also J3.UF8, R20.1; no longer U$9.UF8
- net SCL9_A: now also J2.LE8, R27.1; no longer U$10.LE8
- net SCL9_B: now also J3.LD8, R17.1; no longer U$9.LD8
- net SCL_RAW: now also SCL_RAW.TP
- net VCC3V3: now also J2.LA3, J2.LB3, J2.LC3, J2.LD3, J2.LE3, J2.LF3, J2.LG3, J2.LH3, J2.UA3, J2.UB3, J2.UC3, J2.UD3, J2.UE3, J2.UF3, J2.UG3, J2.UH3, J3.LA3, J3.LB3, J3.LC3, J3.LD3, J3.LE3, J3.LF3, J3.LG3, J3.LH3, J3.UA3, J3.UB3, J3.UC3, J3.UD3, J3.UE3, J3.UF3, J3.UG3, J3.UH3, VCC3V3_TP.TP; no longer U$1.50, U$10.LA3, U$10.LB3, U$10.LC3, U$10.LD3, U$10.LE3, U$10.LF3, U$10.LG3, U$10.LH3, U$10.UA3, U$10.UB3, U$10.UC3, U$10.UD3, U$10.UE3, U$10.UF3, U$10.UG3, U$10.UH3, U$9.LA3, U$9.LB3, U$9.LC3, U$9.LD3, U$9.LE3, U$9.LF3, U$9.LG3, U$9.LH3, U$9.UA3, U$9.UB3, U$9.UC3, U$9.UD3, U$9.UE3, U$9.UF3, U$9.UG3, U$9.UH3
- net VCC5V: now also VCC5V_TP.TP
- net VDD_3V3EXP: now also U$1.50
Routing:
- net GND: track 0.00 -> 684.5 mm, vias 0 -> 78
- net PWM14: track 0.00 -> 273.0 mm, vias 0 -> 4
- net VCC3V3: track 739.4 -> 1008.0 mm, vias 38 -> 37
- net PWM15: track 0.00 -> 267.6 mm, vias 0 -> 4
- net PWM12: track 0.00 -> 261.6 mm, vias 0 -> 4
- net PWM13: track 0.00 -> 255.6 mm, vias 0 -> 4
- net PWM10: track 0.00 -> 247.0 mm, vias 0 -> 4
- net PWM11: track 0.00 -> 238.5 mm, vias 0 -> 4
- net PWM8: track 0.00 -> 224.3 mm, vias 0 -> 4
- net PWM9: track 0.00 -> 218.9 mm, vias 0 -> 4
- net PWM6: track 0.00 -> 203.7 mm, vias 0 -> 4
- net RST: track 737.8 -> 925.2 mm, vias 24 -> 25
- net PWM7: track 0.00 -> 181.7 mm, vias 0 -> 4
- net PWM4: track 0.00 -> 175.3 mm, vias 0 -> 4
- net PWM5: track 0.00 -> 166.0 mm, vias 0 -> 4
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- added copper zone on layer 1, net BIRD1
- added copper zone on layer 1, net GND
- removed copper zone on layer 16, net BIRD1
Other:
- board size 132 x 144 mm -> 134 x 145.5 mm
- board text added: "Burning Man 2015"
- board text added: "CABLES"
- board text added: "CROSSOVER"
- board text added: "Justin Day & Max Henstell"
- board text added: "Keep It Locked"
- board text added: "NO"
- board text added: "Rev B 2014"
- board text removed: "Rev A 2014"

Commit message: Rev B done
Routing:
- net GND: track 684.5 -> 115.1 mm
- net VCC3V3: track 1008.0 -> 755.4 mm, vias 37 -> 38
- net RST: track 925.2 -> 743.7 mm
- net DC: track 791.6 -> 753.6 mm
- net BL-1-2: track 46.9 -> 20.2 mm
- net BL-3-1: track 47.1 -> 21.6 mm
- net BL-11-1: track 44.2 -> 20.5 mm
- net BL-0-2: track 41.2 -> 20.6 mm
- net BL-15-1: track 34.2 -> 15.0 mm
- net PWM13: track 255.6 -> 237.5 mm
- net PWM11: track 238.5 -> 220.6 mm
- net PWM10: track 247.0 -> 229.1 mm
- net PWM9: track 218.9 -> 201.2 mm
- net PWM15: track 267.6 -> 251.3 mm
- net PWM12: track 261.6 -> 246.1 mm
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
Commit message: Oops, adding resistors
Parts:
- added R34, R35, R36, R37, R38, R39, R40, R41: (no value), SparkFun-Passives:0603-RES
Connections:
- net GND: now also R34.2, R35.2, R36.2, R37.2, R38.2, R39.2, R40.2, R41.2
- net SCL0_A: now also R34.1
- net SCL11_A: now also R39.1
- net SCL14_A: now also R40.1
- net SCL15_A: now also R41.1
- net SCL1_A: now also R35.1
- net SCL4_A: now also R36.1
- net SCL5_A: now also R37.1
- net SCL8_A: now also R38.1
Routing:
- net GND: track 115.1 -> 128.5 mm, vias 78 -> 86
- net SCL1_A: track 63.3 -> 59.6 mm
- net SCL11_A: track 40.2 -> 43.7 mm
- net SCL14_A: track 32.4 -> 35.5 mm
- net SCL0_A: track 69.7 -> 67.8 mm
- net DC: track 753.6 -> 755.1 mm
- net SCL4_A: track 57.4 -> 56.0 mm
- net SCL15_A: track 30.1 -> 31.2 mm
- net SCL5_A: track 51.0 -> 51.7 mm
