File: Hardware/tft.sch (EAGLE design)
At the start: 11 parts, among them J1 RJ45-8P8C, J2 40PINFPCM4-1734839-0

Commit message: Finished new tft board
Parts:
- removed H1: MOUNT-HOLE3.0, holes:MOUNT-HOLE3.0
- removed J2: 40PINFPCM4-1734839-0, adafruit:40PINFPCM4-1734839-0
- added U$1: XF2M-4015-WONKY, cape:XF2M-4015-WONKY
- R1, R2, R3, R4: device SparkFun-Passives:RESISTOR0805-RES -> SparkFun-Resistors:RESISTOR0603
Connections:
- net BACKLIGHT: now also J1.6, U$1G$34.MS, U$1G$35.MS, U$1G$36.MS; no longer J1.3, J2-33.MS
- net DATA: now also J1.1, U$1G$13.MS; no longer J1.8, J2-13.MS
- net DC: now also J1.4, U$1G$11.MS; no longer J1.5, J2-11.MS
- net GND: now also U$1G$16.MS, U$1G$37.MS, U$1G$38.MS, U$1G$5.MS, U$1G$9.MS; no longer J2-16.MS, J2-34.MS, J2-35.MS, J2-36.MS, J2-37.MS, J2-38.MS, J2-5.MS, J2-9.MS
- net RST: now also J1.5, U$1G$15.MS; no longer J1.4, J2-15.MS
- net SCK: now also J1.8, U$1G$10.MS; no longer J1.1, J2-10.MS
- net VCC3V3: now also J1.3, U$1G$33.MS, U$1G$39.MS, U$1G$40.MS, U$1G$6.MS, U$1G$7.MS; no longer J1.6, J2-39.MS, J2-40.MS, J2-6.MS, J2-7.MS
