File: Hardware/cape-c.sch (EAGLE design)
At the start: 90 parts, among them IC1 74VHC541, IC2 74VHC541, IC3 74VHC541, IC4 74VHC541, IC5 74VHC541, IC6 74VHC541, IC7 74VHC541, IC8 74VHC541, IC9 74VHC541, J1 MOLEX-P4, J2 RJ45-8P8C-16FCI-16, J3 RJ45-8P8C-16FCI-16, Q1 N-MOSFET-DUALSO8, Q10 N-MOSFET-DUALSO8, Q11 N-MOSFET-DUALSO8, Q12 N-MOSFET-DUALSO8, Q13 N-MOSFET-DUALSO8, Q14 N-MOSFET-DUALSO8, Q15 N-MOSFET-DUALSO8, Q16 N-MOSFET-DUALSO8, Q2 N-MOSFET-DUALSO8, Q3 N-MOSFET-DUALSO8, Q4 N-MOSFET-DUALSO8, Q5 N-MOSFET-DUALSO8, Q6 N-MOSFET-DUALSO8, Q7 N-MOSFET-DUALSO8, Q8 N-MOSFET-DUALSO8, Q9 N-MOSFET-DUALSO8

Commit message: Replaced 5v rail with 3.3v rail (fixes #13)
Parts:
- removed VCC5V_TP: PTR1TP15R, tenna_avr_AD7021_v0_9_shrink:PTR1TP15R
- C1, C2, C20, C21, C3, C4, C5, C6, C7: value 1uF -> 0.1uF
Connections:
- removed net VCC5V: C1.1, C2.1, C20.1, C21.1, C3.1, C4.1, C5.1, C6.1, C7.1, IC1.G1, IC1.VCC, IC2.G1, IC2.VCC, IC3.G1, IC3.VCC, IC4.G1, IC4.VCC, IC5.G1, IC5.VCC, IC6.G1, IC6.VCC, IC7.G1, IC7.VCC, IC8.G1, IC8.VCC, IC9.G1, IC9.VCC, U$1.VDD_5V@1, U$1.VDD_5V@2, VCC5V_TP.TP
- net VCC3V3: now also C1.1, C2.1, C20.1, C21.1, C3.1, C4.1, C5.1, C6.1, C7.1, IC1.G1, IC1.VCC, IC2.G1, IC2.VCC, IC3.G1, IC3.VCC, IC4.G1, IC4.VCC, IC5.G1, IC5.VCC, IC6.G1, IC6.VCC, IC7.G1, IC7.VCC, IC8.G1, IC8.VCC, IC9.G1, IC9.VCC
